File: pcb/interfacez_r1.sch (EAGLE design)
At the start: 128 parts, among them IC10 74LCX245FT, IC11 74LCX245FT, IC2 EP4CE6E22C8N, IC3 74LCX245FT, IC4 74LCX245FT, IC5 MP2233DJ, IC6 MP2233DJ, IC7 CH330N, IC8 MIC5504-2.5YM5-TR, IC9 MT48LC64M4A2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

Commit message: Sync - base stuff working
Connections:
- net XA0 renamed ZX_A11
- net XA1 renamed ZX_A10
- net XA10 renamed ZX_A1
- net XA11 renamed ZX_A0
- net XA12 renamed ZX_A12
- net XA13 renamed ZX_A13
- net XA14 renamed ZX_A14
- net XA15 renamed ZX_A15
- net XA2 renamed ZX_A9
- net XA3 renamed ZX_A8
- net XA4 renamed ZX_A4
- net XA5 renamed ZX_A5
- net XA6 renamed ZX_A6
- net XA7 renamed ZX_A7
- net XA8 renamed ZX_A3
- net XA9 renamed ZX_A2
Changed lines of the file:
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@@
 <layer number="91" name="Nets" color="2" fill="1" visible="yes" active="yes"/>
 <layer number="92" name="Busses" color="1" fill="1" visible="yes" active="yes"/>
-<layer number="93" name="Pins" color="2" fill="1" visible="yes" active="yes"/>
+<layer number="93" name="Pins" color="2" fill="1" visible="no" active="yes"/>
 <layer number="94" name="Symbols" color="4" fill="1" visible="yes" active="yes"/>
 <layer number="95" name="Names" color="7" fill="1" visible="yes" active="yes"/>
@@
 </segment>
 </net>
-<net name="XA15" class="0">
-<segment>
-<label x="330.2" y="170.18" size="1.778" layer="95"/>
-<pinref part="IC10" gate="A" pin="B1"/>
-<wire x1="327.66" y1="170.18" x2="345.44" y2="170.18" width="0.1524" layer="91"/>
-<junction x="327.66" y="170.18"/>
-</segment>
-<segment>
-<pinref part="IC2" gate="G$1" pin="__IO_10"/>
-<wire x1="477.52" y1="386.08" x2="467.36" y2="386.08" width="0.1524" layer="91"/>
-<label x="467.36" y="386.08" size="1.778" layer="95"/>
-</segment>
-</net>
-<net name="XA14" class="0">
+<net name="ZX_A14" class="0">
 <segment>
 <wire x1="345.44" y1="167.64" x2="327.66" y2="167.64" width="0.1524" layer="91"/>
@@
 </segment>
 </net>
-<net name="XA13" class="0">
+<net name="ZX_A13" class="0">
 <segment>
 <label x="330.2" y="165.1" size="1.778" layer="95"/>
@@
 </segment>
 </net>
-<net name="XA12" class="0">
+<net name="ZX_A12" class="0">
 <segment>
 <wire x1="345.44" y1="162.56" x2="327.66" y2="162.56" width="0.1524" layer="91"/>
@@
 </segment>
 </net>
-<net name="XA11" class="0">
+<net name="ZX_A0" class="0">
 <segment>
 <label x="330.2" y="160.02" size="1.778" layer="95"/>
@@
 </segment>
 </net>
-<net name="XA10" class="0">
+<net name="ZX_A1" class="0">
 <segment>
 <wire x1="345.44" y1="157.48" x2="327.66" y2="157.48" width="0.1524" layer="91"/>
@@
 </segment>
 </net>
-<net name="XA9" class="0">
+<net name="ZX_A2" class="0">
 <segment>
 <label x="330.2" y="154.94" size="1.778" layer="95"/>
@@
 </segment>
 </net>
-<net name="XA8" class="0">
+<net name="ZX_A3" class="0">
 <segment>
 <wire x1="345.44" y1="152.4" x2="327.66" y2="152.4" width="0.1524" layer="91"/>
@@
 </segment>
 </net>
-<net name="XA0" class="0">
+<net name="ZX_A11" class="0">
 <segment>
 <label x="330.2" y="104.14" size="1.778" layer="95"/>
@@
 </segment>
 </net>
-<net name="XA1" class="0">
+<net name="ZX_A10" class="0">
 <segment>
 <label x="330.2" y="106.68" size="1.778" layer="95"/>
@@
 </segment>
 </net>
-<net name="XA2" class="0">
+<net name="ZX_A9" class="0">
 <segment>
 <label x="330.2" y="109.22" size="1.778" layer="95"/>
@@
 </segment>
 </net>
-<net name="XA3" class="0">
+<net name="ZX_A8" class="0">
 <segment>
 <label x="330.2" y="111.76" size="1.778" layer="95"/>
@@
 </segment>
 </net>
-<net name="XA4" class="0">
+<net name="ZX_A4" class="0">
 <segment>
 <label x="330.2" y="114.3" size="1.778" layer="95"/>
@@
 </segment>
 </net>
-<net name="XA5" class="0">
+<net name="ZX_A5" class="0">
 <segment>
 <label x="330.2" y="116.84" size="1.778" layer="95"/>
@@
 </segment>
 </net>
-<net name="XA6" class="0">
+<net name="ZX_A6" class="0">
 <segment>
 <label x="330.2" y="119.38" size="1.778" layer="95"/>
@@
 </segment>
 </net>
-<net name="XA7" class="0">
+<net name="ZX_A7" class="0">
 <segment>
 <label x="330.2" y="121.92" size="1.778" layer="95"/>
@@
 </segment>
 </net>
+<net name="ZX_A15" class="0">
+<segment>
+<label x="330.2" y="170.18" size="1.778" layer="95"/>
+<pinref part="IC10" gate="A" pin="B1"/>
+<wire x1="327.66" y1="170.18" x2="345.44" y2="170.18" width="0.1524" layer="91"/>
+<junction x="327.66" y="170.18"/>
+</segment>
+<segment>
+<pinref part="IC2" gate="G$1" pin="__IO_10"/>
+<wire x1="477.52" y1="386.08" x2="467.36" y2="386.08" width="0.1524" layer="91"/>
+<label x="467.36" y="386.08" size="1.778" layer="95"/>
+</segment>
+</net>
