File: pcb/interfacez_r1.brd (EAGLE design)
At the start: 80 x 50 mm, 128 parts, among them IC10 74LCX245FT, IC11 74LCX245FT, IC2 EP4CE6E22C8N, IC3 74LCX245FT, IC4 74LCX245FT, IC5 MP2233DJ, IC6 MP2233DJ, IC7 CH330N, IC8 MIC5504-2.5YM5-TR, IC9 MT48LC64M4A2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

Commit message: Sync - base stuff working
Connections:
- net XA0 renamed ZX_A11
- net XA1 renamed ZX_A10
- net XA10 renamed ZX_A1
- net XA11 renamed ZX_A0
- net XA12 renamed ZX_A12
- net XA13 renamed ZX_A13
- net XA14 renamed ZX_A14
- net XA15 renamed ZX_A15
- net XA2 renamed ZX_A9
- net XA3 renamed ZX_A8
- net XA4 renamed ZX_A4
- net XA5 renamed ZX_A5
- net XA6 renamed ZX_A6
- net XA7 renamed ZX_A7
- net XA8 renamed ZX_A3
- net XA9 renamed ZX_A2
Changed lines of the file:
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@@
 <grid distance="0.5" unitdist="mm" unit="mm" style="lines" multiple="1" display="no" altdistance="0.05" altunitdist="mm" altunit="mm"/>
 <layers>
-<layer number="1" name="Top" color="4" fill="1" visible="yes" active="yes"/>
+<layer number="1" name="Top" color="4" fill="1" visible="no" active="yes"/>
 <layer number="2" name="Route2" color="1" fill="3" visible="no" active="no"/>
 <layer number="3" name="Route3" color="4" fill="3" visible="no" active="no"/>
 <layer number="14" name="Route14" color="1" fill="6" visible="no" active="no"/>
 <layer number="15" name="Route15" color="4" fill="6" visible="no" active="no"/>
-<layer number="16" name="Bottom" color="1" fill="1" visible="no" active="yes"/>
+<layer number="16" name="Bottom" color="1" fill="1" visible="yes" active="yes"/>
 <layer number="17" name="Pads" color="2" fill="1" visible="no" active="yes"/>
 <layer number="18" name="Vias" color="2" fill="1" visible="yes" active="yes"/>
-<layer number="19" name="Unrouted" color="6" fill="1" visible="no" active="yes"/>
+<layer number="19" name="Unrouted" color="6" fill="1" visible="yes" active="yes"/>
 <layer number="20" name="Dimension" color="15" fill="1" visible="no" active="yes"/>
-<layer number="21" name="tPlace" color="7" fill="1" visible="yes" active="yes"/>
+<layer number="21" name="tPlace" color="7" fill="1" visible="no" active="yes"/>
 <layer number="22" name="bPlace" color="7" fill="1" visible="no" active="yes"/>
-<layer number="23" name="tOrigins" color="15" fill="1" visible="yes" active="yes"/>
+<layer number="23" name="tOrigins" color="15" fill="1" visible="no" active="yes"/>
 <layer number="24" name="bOrigins" color="15" fill="1" visible="no" active="yes"/>
-<layer number="25" name="tNames" color="7" fill="1" visible="yes" active="yes"/>
+<layer number="25" name="tNames" color="7" fill="1" visible="no" active="yes"/>
 <layer number="26" name="bNames" color="7" fill="1" visible="no" active="yes"/>
 <layer number="27" name="tValues" color="7" fill="1" visible="no" active="yes"/>
@@
 <layer number="46" name="Milling" color="3" fill="1" visible="no" active="yes"/>
 <layer number="47" name="Measures" color="7" fill="1" visible="no" active="yes"/>
-<layer number="48" name="Document" color="7" fill="1" visible="yes" active="yes"/>
+<layer number="48" name="Document" color="7" fill="1" visible="no" active="yes"/>
 <layer number="49" name="Reference" color="7" fill="1" visible="no" active="yes"/>
 <layer number="50" name="dxf" color="7" fill="1" visible="no" active="no"/>
-<layer number="51" name="tDocu" color="7" fill="1" visible="yes" active="yes"/>
+<layer number="51" name="tDocu" color="7" fill="1" visible="no" active="yes"/>
 <layer number="52" name="bDocu" color="7" fill="1" visible="no" active="yes"/>
 <layer number="53" name="tGND_GNDA" color="7" fill="1" visible="no" active="no"/>
@@
 <contactref element="IC3" pad="19"/>
 </signal>
-<signal name="XA15">
-<wire x1="34.95" y1="24.2" x2="34.95" y2="22.8" width="0.1524" layer="1"/>
-<via x="34.95" y="22.8" extent="1-16" drill="0.3"/>
-<wire x1="34.95" y1="22.8" x2="34.95" y2="20.1" width="0.1524" layer="16"/>
-<wire x1="37.375" y1="18.0178" x2="37.375" y2="18.575" width="0.1524" layer="1"/>
-<wire x1="37.375" y1="18.575" x2="37.05" y2="18.95" width="0.1524" layer="1"/>
-<wire x1="37.05" y1="18.95" x2="35.15" y2="18.95" width="0.1524" layer="1"/>
-<wire x1="35.15" y1="18.95" x2="34.95" y2="19.15" width="0.1524" layer="1"/>
-<via x="34.95" y="20.1" extent="1-16" drill="0.3"/>
-<wire x1="34.95" y1="20.1" x2="34.95" y2="19.15" width="0.1524" layer="1"/>
-<contactref element="IC2" pad="28"/>
-<wire x1="40.187" y1="28.27" x2="39.02" y2="28.27" width="0.1524" layer="1"/>
-<wire x1="39.02" y1="28.27" x2="34.95" y2="24.2" width="0.1524" layer="1"/>
-<contactref element="IC10" pad="18"/>
-</signal>
-<signal name="XA14">
+<signal name="ZX_A14">
 <wire x1="35.65" y1="24.35" x2="35.65" y2="23.55" width="0.1524" layer="1"/>
 <via x="35.65" y="23.55" extent="1-16" drill="0.3"/>
@@
 <contactref element="IC10" pad="17"/>
 </signal>
-<signal name="XA13">
+<signal name="ZX_A13">
 <wire x1="36.25" y1="24.4" x2="36.25" y2="22.85" width="0.1524" layer="1"/>
 <via x="36.25" y="22.85" extent="1-16" drill="0.3"/>
@@
 <contactref element="IC10" pad="16"/>
 </signal>
-<signal name="XA12">
+<signal name="ZX_A12">
 <contactref element="IC2" pad="32"/>
 <via x="37" y="24.25" extent="1-16" drill="0.3"/>
@@
 <contactref element="IC10" pad="15"/>
 </signal>
-<signal name="XA11">
+<signal name="ZX_A0">
 <contactref element="IC2" pad="33"/>
 <via x="37.6" y="23.45" extent="1-16" drill="0.3"/>
@@
 <contactref element="IC10" pad="14"/>
 </signal>
-<signal name="XA10">
+<signal name="ZX_A1">
 <contactref element="IC2" pad="34"/>
 <wire x1="40.187" y1="25.27" x2="39.17" y2="25.27" width="0.1524" layer="1"/>
@@
 <contactref element="IC10" pad="13"/>
 </signal>
-<signal name="XA9">
+<signal name="ZX_A2">
 <contactref element="IC2" pad="38"/>
 <wire x1="42.675" y1="22.282" x2="42.675" y2="21.275" width="0.1524" layer="1"/>
@@
 <contactref element="IC10" pad="12"/>
 </signal>
-<signal name="XA8">
+<signal name="ZX_A3">
 <contactref element="IC2" pad="39"/>
 <wire x1="43.175" y1="22.282" x2="43.175" y2="20.725" width="0.1524" layer="1"/>
@@
 <contactref element="IC10" pad="11"/>
 </signal>
-<signal name="XA0">
+<signal name="ZX_A11">
 <contactref element="IC2" pad="75"/>
 <wire x1="61.663" y1="25.27" x2="62.78" y2="25.27" width="0.1524" layer="1"/>
@@
 <wire x1="67.9822" y1="19.475" x2="66.475" y2="19.475" width="0.1524" layer="1"/>
 </signal>
-<signal name="XA1">
+<signal name="ZX_A10">
 <contactref element="IC2" pad="74"/>
 <wire x1="61.663" y1="24.77" x2="62.63" y2="24.77" width="0.1524" layer="1"/>
@@
 <wire x1="67.9822" y1="18.825" x2="66.475" y2="18.825" width="0.1524" layer="1"/>
 </signal>
-<signal name="XA2">
+<signal name="ZX_A9">
 <contactref element="IC2" pad="73"/>
 <wire x1="61.663" y1="24.27" x2="62.48" y2="24.27" width="0.1524" layer="1"/>
@@
 <wire x1="67.9822" y1="18.175" x2="66.475" y2="18.175" width="0.1524" layer="1"/>
 </signal>
-<signal name="XA3">
+<signal name="ZX_A8">
 <contactref element="IC2" pad="72"/>
 <wire x1="59.675" y1="22.282" x2="59.675" y2="21.525" width="0.1524" layer="1"/>
@@
 <wire x1="67.9822" y1="17.525" x2="63.675" y2="17.525" width="0.1524" layer="1"/>
 </signal>
-<signal name="XA4">
+<signal name="ZX_A4">
 <contactref element="IC2" pad="71"/>
 <wire x1="59.175" y1="22.282" x2="59.175" y2="21.425" width="0.1524" layer="1"/>
@@
 <wire x1="67.9822" y1="16.875" x2="63.725" y2="16.875" width="0.1524" layer="1"/>
 </signal>
-<signal name="XA5">
+<signal name="ZX_A5">
 <contactref element="IC2" pad="70"/>
 <wire x1="58.675" y1="22.282" x2="58.675" y2="21.275" width="0.1524" layer="1"/>
@@
 <wire x1="67.9822" y1="16.225" x2="63.725" y2="16.225" width="0.1524" layer="1"/>
 </signal>
-<signal name="XA6">
+<signal name="ZX_A6">
 <contactref element="IC2" pad="69"/>
 <wire x1="58.175" y1="22.282" x2="58.175" y2="21.125" width="0.1524" layer="1"/>
@@
 <wire x1="67.9822" y1="15.575" x2="63.725" y2="15.575" width="0.1524" layer="1"/>
 </signal>
-<signal name="XA7">
+<signal name="ZX_A7">
 <contactref element="IC2" pad="68"/>
 <wire x1="57.675" y1="22.282" x2="57.675" y2="20.975" width="0.1524" layer="1"/>
@@
 <wire x1="47.85" y1="46.25" x2="49.1" y2="46.25" width="0.1524" layer="1"/>
 </signal>
+<signal name="ZX_A15">
+<contactref element="IC10" pad="18"/>
+<wire x1="34.95" y1="24.2" x2="34.95" y2="22.8" width="0.1524" layer="1"/>
+<via x="34.95" y="22.8" extent="1-16" drill="0.3"/>
+<wire x1="34.95" y1="22.8" x2="34.95" y2="20.1" width="0.1524" layer="16"/>
+<wire x1="37.375" y1="18.575" x2="37.05" y2="18.95" width="0.1524" layer="1"/>
+<wire x1="37.05" y1="18.95" x2="35.15" y2="18.95" width="0.1524" layer="1"/>
+<wire x1="35.15" y1="18.95" x2="34.95" y2="19.15" width="0.1524" layer="1"/>
+<via x="34.95" y="20.1" extent="1-16" drill="0.3"/>
+<wire x1="34.95" y1="20.1" x2="34.95" y2="19.15" width="0.1524" layer="1"/>
+<contactref element="IC2" pad="28"/>
+<wire x1="40.187" y1="28.27" x2="39.02" y2="28.27" width="0.1524" layer="1"/>
+<wire x1="39.02" y1="28.27" x2="34.95" y2="24.2" width="0.1524" layer="1"/>
+<wire x1="37.375" y1="18.575" x2="37.375" y2="18.0178" width="0.1524" layer="1"/>
+</signal>
 </signals>
