File: pcb/interfacez_r2.brd (EAGLE design)
At the start: 80 x 50 mm, 137 parts, among them IC10 74LCX245FT, IC11 74LCX245FT, IC2 EP4CE6E22C8N, IC3 74LCX245FT, IC4 74LCX245FT, IC5 MP2233DJ, IC6 MP2233DJ, IC7 CH330N, IC8 MIC5504-2.5YM5-TR, IC9 MT48LC64M4A2, Q1 BSS123, Q2 BSS123, Q3 BSS123, Q4 BSS84, Q5 BSS84, U1 ESP-WROOM-32, U2 EPCS16

Commit message: Preliminary version for SNA loading
Connections:
- net XA0 renamed ZX_A11
- net XA1 renamed ZX_A10
- net XA10 renamed ZX_A1
- net XA11 renamed ZX_A0
- net XA12 renamed ZX_A12
- net XA13 renamed ZX_A13
- net XA14 renamed ZX_A14
- net XA15 renamed ZX_A15
- net XA2 renamed ZX_A9
- net XA3 renamed ZX_A8
- net XA4 renamed ZX_A4
- net XA5 renamed ZX_A5
- net XA6 renamed ZX_A6
- net XA7 renamed ZX_A7
- net XA8 renamed ZX_A3
- net XA9 renamed ZX_A2
Changed lines of the file:
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@@
 <contactref element="IC3" pad="19"/>
 </signal>
-<signal name="XA15">
+<signal name="ZX_A15">
 <wire x1="34.95" y1="24.2" x2="34.95" y2="22.8" width="0.1524" layer="1"/>
 <via x="34.95" y="22.8" extent="1-16" drill="0.3"/>
@@
 <contactref element="IC10" pad="18"/>
 </signal>
-<signal name="XA14">
+<signal name="ZX_A14">
 <wire x1="35.65" y1="24.35" x2="35.65" y2="23.55" width="0.1524" layer="1"/>
 <via x="35.65" y="23.55" extent="1-16" drill="0.3"/>
@@
 <contactref element="IC10" pad="17"/>
 </signal>
-<signal name="XA13">
+<signal name="ZX_A13">
 <wire x1="36.25" y1="24.4" x2="36.25" y2="22.85" width="0.1524" layer="1"/>
 <via x="36.25" y="22.85" extent="1-16" drill="0.3"/>
@@
 <contactref element="IC10" pad="16"/>
 </signal>
-<signal name="XA12">
+<signal name="ZX_A12">
 <contactref element="IC2" pad="32"/>
 <via x="37" y="24.25" extent="1-16" drill="0.3"/>
@@
 <contactref element="IC10" pad="15"/>
 </signal>
-<signal name="XA11">
+<signal name="ZX_A0">
 <contactref element="IC2" pad="33"/>
 <via x="37.6" y="23.45" extent="1-16" drill="0.3"/>
@@
 <contactref element="IC10" pad="14"/>
 </signal>
-<signal name="XA10">
+<signal name="ZX_A1">
 <contactref element="IC2" pad="34"/>
 <wire x1="40.187" y1="25.27" x2="39.17" y2="25.27" width="0.1524" layer="1"/>
@@
 <contactref element="IC10" pad="13"/>
 </signal>
-<signal name="XA9">
+<signal name="ZX_A2">
 <contactref element="IC2" pad="38"/>
 <wire x1="42.675" y1="22.282" x2="42.675" y2="21.275" width="0.1524" layer="1"/>
@@
 <contactref element="IC10" pad="12"/>
 </signal>
-<signal name="XA8">
+<signal name="ZX_A3">
 <contactref element="IC2" pad="39"/>
 <wire x1="43.175" y1="22.282" x2="43.175" y2="20.725" width="0.1524" layer="1"/>
@@
 <contactref element="IC10" pad="11"/>
 </signal>
-<signal name="XA0">
+<signal name="ZX_A11">
 <contactref element="IC2" pad="75"/>
 <wire x1="61.663" y1="25.27" x2="62.78" y2="25.27" width="0.1524" layer="1"/>
@@
 <wire x1="67.9822" y1="19.475" x2="66.475" y2="19.475" width="0.1524" layer="1"/>
 </signal>
-<signal name="XA1">
+<signal name="ZX_A10">
 <contactref element="IC2" pad="74"/>
 <wire x1="61.663" y1="24.77" x2="62.63" y2="24.77" width="0.1524" layer="1"/>
@@
 <wire x1="67.9822" y1="18.825" x2="66.475" y2="18.825" width="0.1524" layer="1"/>
 </signal>
-<signal name="XA2">
+<signal name="ZX_A9">
 <contactref element="IC2" pad="73"/>
 <wire x1="61.663" y1="24.27" x2="62.48" y2="24.27" width="0.1524" layer="1"/>
@@
 <wire x1="67.9822" y1="18.175" x2="66.475" y2="18.175" width="0.1524" layer="1"/>
 </signal>
-<signal name="XA3">
+<signal name="ZX_A8">
 <contactref element="IC2" pad="72"/>
 <wire x1="59.675" y1="22.282" x2="59.675" y2="21.525" width="0.1524" layer="1"/>
@@
 <wire x1="67.9822" y1="17.525" x2="63.675" y2="17.525" width="0.1524" layer="1"/>
 </signal>
-<signal name="XA4">
+<signal name="ZX_A4">
 <contactref element="IC2" pad="71"/>
 <wire x1="59.175" y1="22.282" x2="59.175" y2="21.425" width="0.1524" layer="1"/>
@@
 <wire x1="67.9822" y1="16.875" x2="63.725" y2="16.875" width="0.1524" layer="1"/>
 </signal>
-<signal name="XA5">
+<signal name="ZX_A5">
 <contactref element="IC2" pad="70"/>
 <wire x1="58.675" y1="22.282" x2="58.675" y2="21.275" width="0.1524" layer="1"/>
@@
 <wire x1="67.9822" y1="16.225" x2="63.725" y2="16.225" width="0.1524" layer="1"/>
 </signal>
-<signal name="XA6">
+<signal name="ZX_A6">
 <contactref element="IC2" pad="69"/>
 <wire x1="58.175" y1="22.282" x2="58.175" y2="21.125" width="0.1524" layer="1"/>
@@
 <wire x1="67.9822" y1="15.575" x2="63.725" y2="15.575" width="0.1524" layer="1"/>
 </signal>
-<signal name="XA7">
+<signal name="ZX_A7">
 <contactref element="IC2" pad="68"/>
 <wire x1="57.675" y1="22.282" x2="57.675" y2="20.975" width="0.1524" layer="1"/>

Commit message: Preparing for SNA
Parts:
- added Q6: BSS123, transistor-small-signal:SOT23
- C40: value 1uF -> 10uF
Connections:
- removed net ESP_IO25: IC2.137, U1.10
- new net FORCE_NMI: IC2.137, Q6.1
- new net NMI: CONN1.B14, Q6.3
- net GND: now also Q6.2
- net NCONFIG: now also U1.10
Routing:
- net ESP_IO25: track 35.7 -> 0.00 mm, vias 1 -> 0
- net FORCE_NMI: track 0.00 -> 18.6 mm, vias 0 -> 2
- net NMI: track 0.00 -> 2.91 mm
- net A2: track 11.1 -> 13.4 mm
- net A3: track 10.4 -> 12.1 mm
- net A0: track 14.3 -> 14.9 mm

Commit message: Sync - working version with SNAs
Parts:
- removed IC9: MT48LC64M4A2, memory-micron:TSOP54-400
- added C59: 100nF 6.3V, GadgetFactory:0603
- added C61: 4.7uF 6.3V, GadgetFactory:0805
- added IC1: STMPS2141STR, alvie:SOT23-5L
- added Q7: BSS123, transistor-small-signal:SOT23
- added R37, R38: 100K, GadgetFactory:0603
- added R39: 12K, GadgetFactory:0603
- added R40: 820R, GadgetFactory:0603
- added TV26: SP0503BAHT, alvie:SP0503
- added U$2, U$3: LY68L6400SLIT, alvie:SOIC8
- added U$4: USB3300-EZK, alvie:QFN32
- added X1: USB-A-H, con-usb:USB-A-H
- C54: value 100nF 6.3V -> 120uF 6.3V TANT; device GadgetFactory:0603 -> alvie:TANT_CASE_A
- moved C54 126.6 mm to (-6.00, -63.0), flipped to the top, turned to 0 degrees
- moved C53 123.5 mm to (-6.00, -52.0), flipped to the top
- moved C51 114.7 mm to (-6.00, -44.0), flipped to the top, turned to 0 degrees
- moved C52 114.1 mm to (-6.00, -48.0), flipped to the top, turned to 0 degrees
- moved C50 98.6 mm to (-6.00, -40.0), flipped to the top, turned to 0 degrees
- moved C48 22.3 mm to (79.3, 23.1), turned to 90 degrees
- moved C49 10.3 mm to (71.0, 22.8), turned to 90 degrees
- moved C60 6.08 mm to (60.6, 46.5)
- moved CONN1 5.00 mm to (20.9, 1.60)
- moved Q6 0.34 mm to (51.8, 9.85), turned to 180 degrees
Connections:
- new net N$20: R40.2, U$4.4
- new net N$55: C59.1, C61.2, U$4.15, U$4.26
- new net N$57: R39.2, U$4.32
- new net N$58: U$4.29
- new net N$61: U$4.22
- new net N$62: U$4.21
- new net N$63: U$4.20
- new net N$64: U$4.19
- new net N$65: U$4.18
- new net N$66: U$4.17
- new net PE: Q7.2, X1.P$5, X1.P$6
- new net PEN1: IC1.4, Q7.3, R37.1
- new net RAMCLK: U$2.6
- new net RAMD0: U$2.5
- new net RAMD1: U$2.2
- new net RAMD2: U$2.3
- new net RAMD3: U$2.7
- new net RAMNCS: U$2.1
- new net ULPI_1: U$4.23
- new net ULPI_CLK: U$4.28
- new net ULPI_D0: U$4.24
- new net USBHS_DM: TV26.3, U$4.8, X1.D-
- new net USBHS_DP: TV26.2, U$4.7, X1.D+
- new net USBHS_VBUS: C54.PLUS, IC1.1, R40.1, TV26.4, X1.VBUS
- new net USB_FLT: IC1.3, R38.1, U$4.10
- new net USB_PWREN: Q7.1, U$4.3
- new net VCC: U$3.8
- new net VDD3.3: U$4.25
- net +3V3: now also C48.2, C49.2, R38.2, U$2.8, U$4.16, U$4.30, U$4.31, U$4.6; no longer C48.1, C49.1, C54.1, IC9.1, IC9.14, IC9.27, IC9.3, IC9.43, IC9.49, IC9.9
- net +5V: now also IC1.5, R37.2
- net GND: now also C48.1, C49.1, C54.MINUS, C59.2, C61.1, IC1.2, R39.1, TV26.1, U$2.4, U$3.4, U$4.1, U$4.2, U$4.EXP, X1.GND; no longer C48.2, C49.2, C54.2, IC9.12, IC9.28, IC9.41, IC9.46, IC9.52, IC9.54, IC9.6
- net SD_A0: no longer IC9.23
- net SD_A1: no longer IC9.24
- net SD_A10: no longer IC9.22
- net SD_A11: no longer IC9.35
- net SD_A12: no longer IC9.36
- net SD_A2: no longer IC9.25
- net SD_A3: no longer IC9.26
- net SD_A4: no longer IC9.29
- net SD_A5: no longer IC9.30
- net SD_A6: no longer IC9.31
- net SD_A7: no longer IC9.32
- net SD_A8: no longer IC9.33
- net SD_A9: no longer IC9.34
- net SD_BA0: no longer IC9.20
- net SD_BA1: no longer IC9.21
- net SD_CK: no longer IC9.38
- net SD_CKE: no longer IC9.37
- net SD_CS: no longer IC9.19
- net SD_DQ0: no longer IC9.2
- net SD_DQ1: no longer IC9.4
- net SD_DQ2: no longer IC9.5
- net SD_DQ3: no longer IC9.7
- net SD_DQ4: no longer IC9.8
- net SD_DQ5: no longer IC9.10
- net SD_DQ6: no longer IC9.11
- net SD_DQ7: no longer IC9.13
- net SD_DQMH: no longer IC9.39
- net SD_NCAS: no longer IC9.17
- net SD_NRAS: no longer IC9.18
- net SD_NWE: no longer IC9.16
Routing:
- net SD_DQMH: track 46.9 -> 0.00 mm
- net SD_A9: track 46.5 -> 0.00 mm
- net SD_CK: track 46.4 -> 0.00 mm
- net SD_CKE: track 45.9 -> 0.00 mm
- net SD_A8: track 45.8 -> 0.00 mm
- net SD_A12: track 45.3 -> 0.00 mm
- net SD_A11: track 44.8 -> 0.00 mm
- net SD_A7: track 24.5 -> 0.00 mm
- net SD_A6: track 23.3 -> 0.00 mm
- net SD_A5: track 22.0 -> 0.00 mm
- net SD_A4: track 21.8 -> 0.00 mm
- net FORCE_NMI: track 18.6 -> 37.1 mm, vias 2 -> 4
- net SD_DQ0: track 16.4 -> 0.00 mm
- net SD_DQ5: track 15.2 -> 0.00 mm
- net SD_DQ3: track 15.2 -> 0.00 mm
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Other:
- board size 80 x 50 mm -> 85 x 50 mm
