File: pcb/interfacez_r2.sch (EAGLE design)
At the start: 137 parts, among them IC10 74LCX245FT, IC11 74LCX245FT, IC2 EP4CE6E22C8N, IC3 74LCX245FT, IC4 74LCX245FT, IC5 MP2233DJ, IC6 MP2233DJ, IC7 CH330N, IC8 MIC5504-2.5YM5-TR, IC9 MT48LC64M4A2, Q1 BSS123, Q2 BSS123, Q3 BSS123, Q4 BSS84, Q5 BSS84, U1 ESP-WROOM-32, U2 EPCS16

Commit message: Preliminary version for SNA loading
Connections:
- net XA0 renamed ZX_A11
- net XA1 renamed ZX_A10
- net XA10 renamed ZX_A1
- net XA11 renamed ZX_A0
- net XA12 renamed ZX_A12
- net XA13 renamed ZX_A13
- net XA14 renamed ZX_A14
- net XA15 renamed ZX_A15
- net XA2 renamed ZX_A9
- net XA3 renamed ZX_A8
- net XA4 renamed ZX_A4
- net XA5 renamed ZX_A5
- net XA6 renamed ZX_A6
- net XA7 renamed ZX_A7
- net XA8 renamed ZX_A3
- net XA9 renamed ZX_A2
Changed lines of the file:
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@@
 <layer number="91" name="Nets" color="2" fill="1" visible="yes" active="yes"/>
 <layer number="92" name="Busses" color="1" fill="1" visible="yes" active="yes"/>
-<layer number="93" name="Pins" color="2" fill="1" visible="yes" active="yes"/>
+<layer number="93" name="Pins" color="2" fill="1" visible="no" active="yes"/>
 <layer number="94" name="Symbols" color="4" fill="1" visible="yes" active="yes"/>
 <layer number="95" name="Names" color="7" fill="1" visible="yes" active="yes"/>
@@
 </segment>
 </net>
-<net name="XA15" class="0">
+<net name="ZX_A15" class="0">
 <segment>
 <label x="330.2" y="170.18" size="1.778" layer="95"/>
@@
 </segment>
 </net>
-<net name="XA14" class="0">
+<net name="ZX_A14" class="0">
 <segment>
 <wire x1="345.44" y1="167.64" x2="327.66" y2="167.64" width="0.1524" layer="91"/>
@@
 </segment>
 </net>
-<net name="XA13" class="0">
+<net name="ZX_A13" class="0">
 <segment>
 <label x="330.2" y="165.1" size="1.778" layer="95"/>
@@
 </segment>
 </net>
-<net name="XA12" class="0">
+<net name="ZX_A12" class="0">
 <segment>
 <wire x1="345.44" y1="162.56" x2="327.66" y2="162.56" width="0.1524" layer="91"/>
@@
 </segment>
 </net>
-<net name="XA11" class="0">
+<net name="ZX_A0" class="0">
 <segment>
 <label x="330.2" y="160.02" size="1.778" layer="95"/>
@@
 </segment>
 </net>
-<net name="XA10" class="0">
+<net name="ZX_A1" class="0">
 <segment>
 <wire x1="345.44" y1="157.48" x2="327.66" y2="157.48" width="0.1524" layer="91"/>
@@
 </segment>
 </net>
-<net name="XA9" class="0">
+<net name="ZX_A2" class="0">
 <segment>
 <label x="330.2" y="154.94" size="1.778" layer="95"/>
@@
 </segment>
 </net>
-<net name="XA8" class="0">
+<net name="ZX_A3" class="0">
 <segment>
 <wire x1="345.44" y1="152.4" x2="327.66" y2="152.4" width="0.1524" layer="91"/>
@@
 </segment>
 </net>
-<net name="XA0" class="0">
+<net name="ZX_A11" class="0">
 <segment>
 <label x="330.2" y="104.14" size="1.778" layer="95"/>
@@
 </segment>
 </net>
-<net name="XA1" class="0">
+<net name="ZX_A10" class="0">
 <segment>
 <label x="330.2" y="106.68" size="1.778" layer="95"/>
@@
 </segment>
 </net>
-<net name="XA2" class="0">
+<net name="ZX_A9" class="0">
 <segment>
 <label x="330.2" y="109.22" size="1.778" layer="95"/>
@@
 </segment>
 </net>
-<net name="XA3" class="0">
+<net name="ZX_A8" class="0">
 <segment>
 <label x="330.2" y="111.76" size="1.778" layer="95"/>
@@
 </segment>
 </net>
-<net name="XA4" class="0">
+<net name="ZX_A4" class="0">
 <segment>
 <label x="330.2" y="114.3" size="1.778" layer="95"/>
@@
 </segment>
 </net>
-<net name="XA5" class="0">
+<net name="ZX_A5" class="0">
 <segment>
 <label x="330.2" y="116.84" size="1.778" layer="95"/>
@@
 </segment>
 </net>
-<net name="XA6" class="0">
+<net name="ZX_A6" class="0">
 <segment>
 <label x="330.2" y="119.38" size="1.778" layer="95"/>
@@
 </segment>
 </net>
-<net name="XA7" class="0">
+<net name="ZX_A7" class="0">
 <segment>
 <label x="330.2" y="121.92" size="1.778" layer="95"/>

Commit message: Preparing for SNA
Parts:
- added Q6: BSS123, transistor-small-signal:BSS123
- C40: value 1uF -> 10uF
Connections:
- removed net ESP_IO25: IC2.__IO_79, U1.IO25
- new net FORCE_NMI: IC2.__IO_79, Q6.G
- new net NMI: CONN1.NMI, Q6.D
- net GND: now also Q6.S
- net NCONFIG: now also U1.IO25
Changed lines of the file:
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@@
 <part name="GND101" library="supply1" deviceset="GND" device=""/>
 <part name="GND102" library="supply1" deviceset="GND" device=""/>
-<part name="C40" library="GadgetFactory" deviceset="C" device="0603" value="1uF"/>
+<part name="C40" library="GadgetFactory" deviceset="C" device="0603" value="10uF"/>
 <part name="GND2" library="supply1" deviceset="GND" device=""/>
 <part name="C37" library="GadgetFactory" deviceset="C" device="0603" value="1uF"/>
@@
 <part name="R33" library="GadgetFactory" deviceset="R" device="0603" value="10K"/>
 <part name="R34" library="GadgetFactory" deviceset="R" device="0603" value="10K"/>
+<part name="Q6" library="transistor-small-signal" deviceset="BSS123" device=""/>
+<part name="GND62" library="supply1" deviceset="GND" device=""/>
 </parts>
 <sheets>
@@
 <instance part="R33" gate="A" x="38.1" y="431.8" rot="R90"/>
 <instance part="R34" gate="A" x="30.48" y="431.8" rot="R90"/>
+<instance part="Q6" gate="G$1" x="99.06" y="129.54"/>
+<instance part="GND62" gate="1" x="99.06" y="119.38"/>
 </instances>
 <busses>
@@
 <wire x1="7.62" y1="342.9" x2="7.62" y2="345.44" width="0.1524" layer="91"/>
 </segment>
+<segment>
+<pinref part="Q6" gate="G$1" pin="S"/>
+<pinref part="GND62" gate="1" pin="GND"/>
+<wire x1="99.06" y1="124.46" x2="99.06" y2="121.92" width="0.1524" layer="91"/>
+</segment>
 </net>
 <net name="N$149" class="0">
@@
 <pinref part="R7" gate="A" pin="1"/>
 </segment>
+<segment>
+<pinref part="U1" gate="G$1" pin="IO25"/>
+<wire x1="33.02" y1="335.28" x2="20.32" y2="335.28" width="0.1524" layer="91"/>
+<label x="20.32" y="335.28" size="1.778" layer="95"/>
+</segment>
 </net>
 <net name="DCLK" class="0">
@@
 </segment>
 </net>
-<net name="ESP_IO25" class="0">
-<segment>
-<pinref part="U1" gate="G$1" pin="IO25"/>
-<wire x1="33.02" y1="335.28" x2="20.32" y2="335.28" width="0.1524" layer="91"/>
-<label x="20.32" y="335.28" size="1.778" layer="95"/>
-</segment>
-<segment>
-<pinref part="IC2" gate="G$1" pin="__IO_79"/>
-<wire x1="505.46" y1="480.06" x2="505.46" y2="492.76" width="0.1524" layer="91"/>
-<label x="505.46" y="482.6" size="1.778" layer="95" rot="R90"/>
-</segment>
-</net>
 <net name="ESP_IO26" class="0">
 <segment>
@@
 </segment>
 </net>
+<net name="FORCE_NMI" class="0">
+<segment>
+<pinref part="Q6" gate="G$1" pin="G"/>
+<wire x1="93.98" y1="127" x2="91.44" y2="127" width="0.1524" layer="91"/>
+<wire x1="91.44" y1="127" x2="91.44" y2="121.92" width="0.1524" layer="91"/>
+<wire x1="91.44" y1="121.92" x2="76.2" y2="121.92" width="0.1524" layer="91"/>
+<label x="76.2" y="121.92" size="1.778" layer="95"/>
+</segment>
+<segment>
+<pinref part="IC2" gate="G$1" pin="__IO_79"/>
+<wire x1="505.46" y1="480.06" x2="505.46" y2="492.76" width="0.1524" layer="91"/>
+<label x="505.46" y="482.6" size="1.778" layer="95" rot="R90"/>
+</segment>
+</net>
+<net name="NMI" class="0">
+<segment>
+<pinref part="Q6" gate="G$1" pin="D"/>
+<wire x1="99.06" y1="134.62" x2="99.06" y2="137.16" width="0.1524" layer="91"/>
+<wire x1="99.06" y1="137.16" x2="78.74" y2="137.16" width="0.1524" layer="91"/>
+<label x="78.74" y="137.16" size="1.778" layer="95"/>
+</segment>
+<segment>
+<pinref part="CONN1" gate="G$1" pin="NMI"/>
+<wire x1="114.3" y1="182.88" x2="104.14" y2="182.88" width="0.1524" layer="91"/>
+<label x="104.14" y="182.88" size="1.778" layer="95"/>
+</segment>
+</net>

Commit message: Sync - working version with SNAs
Parts:
- removed IC9: MT48LC64M4A2, memory-micron:MT48LC64M4A2
- added C59: 100nF 6.3V, GadgetFactory:C0603
- added C61: 4.7uF 6.3V, GadgetFactory:C0805
- added IC1: STMPS2141STR, alvie:STMPS2141STR
- added Q7: BSS123, transistor-small-signal:BSS123
- added R37, R38: 100K, GadgetFactory:R0603
- added R39: 12K, GadgetFactory:R0603
- added R40: 820R, GadgetFactory:R0603
- added TV26: SP0503BAHT, alvie:SP0503BAHT
- added U$2, U$3: LY68L6400SLIT, alvie:LY68L6400SLIT
- added U$4: USB3300-EZK, alvie:USB3300-EZK
- added X1: USB-A-H, con-usb:USB-A-H
- C54: value 100nF 6.3V -> 120uF 6.3V TANT; device GadgetFactory:C0603 -> alvie:TANT_CASE_A
Connections:
- new net N$20: R40A.2, U$4.VBUS
- new net N$55: C59.1, C61.2, U$4.VDD1.8, U$4.VDD1.8@1
- new net N$57: R39A.2, U$4.RBIAS
- new net N$58: U$4.VDDA1.8
- new net N$61: U$4.D2
- new net N$62: U$4.D3
- new net N$63: U$4.D4
- new net N$64: U$4.D5
- new net N$65: U$4.D6
- new net N$66: U$4.D7
- new net PE: Q7.S, X1.SHIELD
- new net PEN1: IC1.NEN, Q7.D, R37A.1
- new net RAMCLK: U$2.SCK
- new net RAMD0: U$2.SI/SIO[0]
- new net RAMD1: U$2.SO/SIO[1]
- new net RAMD2: U$2.SIO[2]
- new net RAMD3: U$2.SIO[3]
- new net RAMNCS: U$2.NCS
- new net ULPI_1: U$4.D1
- new net ULPI_CLK: U$4.XI
- new net ULPI_D0: U$4.D0
- new net USBHS_DM: TV26.B, U$4.DM, X1.D-
- new net USBHS_DP: TV26.A, U$4.DP, X1.D+
- new net USBHS_VBUS: C54.+, IC1.VOUT, R40A.1, TV26.C, X1.VBUS
- new net USB_FLT: IC1.FAULT, R38A.1, U$4.EXTVBUS
- new net USB_PWREN: Q7.G, U$4.CPEN
- net +3V3: now also C48.2, C49.2, R38A.2, U$2.VCC, U$4.REG_EN, U$4.VDD3.3, U$4.VDD3.3@1, U$4.VDD3.3@3; no longer C48.1, C49.1, C54.1, IC9P.VDD@1, IC9P.VDD@2, IC9P.VDD@3, IC9P.VDDQ@1, IC9P.VDDQ@2, IC9P.VDDQ@3, IC9P.VDDQ@4
- net +5V: now also IC1.VIN, R37A.2
- net GND: now also C48.1, C49.1, C54.-, C59.2, C61.1, IC1.GND, R39A.1, TV26.COM, U$2.GND, U$4.GND@1, U$4.GND@2, U$4.PAD, X1.GND; no longer C48.2, C49.2, C54.2, IC9P.VSS@1, IC9P.VSS@2, IC9P.VSS@3, IC9P.VSSQ@1, IC9P.VSSQ@2, IC9P.VSSQ@3, IC9P.VSSQ@4
- net SD_A0: no longer IC9G$1.A0
- net SD_A1: no longer IC9G$1.A1
- net SD_A10: no longer IC9G$1.A10
- net SD_A11: no longer IC9G$1.A11
- net SD_A12: no longer IC9G$1.A12
- net SD_A2: no longer IC9G$1.A2
- net SD_A3: no longer IC9G$1.A3
- net SD_A4: no longer IC9G$1.A4
- net SD_A5: no longer IC9G$1.A5
- net SD_A6: no longer IC9G$1.A6
- net SD_A7: no longer IC9G$1.A7
- net SD_A8: no longer IC9G$1.A8
- net SD_A9: no longer IC9G$1.A9
- net SD_BA0: no longer IC9G$1.BA0
- net SD_BA1: no longer IC9G$1.BA1
- net SD_CK: no longer IC9G$1.CLK
- net SD_CKE: no longer IC9G$1.CKE
- net SD_CS: no longer IC9G$1.\CS
- net SD_DQ0: no longer IC9G$1.DQ0
- net SD_DQ1: no longer IC9G$1.DQ1
- net SD_DQ2: no longer IC9G$1.DQ2
- net SD_DQ3: no longer IC9G$1.DQ3
- net SD_DQ4: no longer IC9G$1.DQ4
- net SD_DQ5: no longer IC9G$1.DQ5
- net SD_DQ6: no longer IC9G$1.DQ6
- net SD_DQ7: no longer IC9G$1.DQ7
- net SD_DQMH: no longer IC9G$1.DQMH
- net SD_NCAS: no longer IC9G$1.!CAS
- net SD_NRAS: no longer IC9G$1.!RAS
- net SD_NWE: no longer IC9G$1.!WE
Other:
- note added: "USB Host connector"
- moved on the sheet: C48, C49, C50, C51, C52, C53, R24, R25, R26
