File: pcb/interfacez_r2_1.brd (EAGLE design)
At the start: 100 x 50 mm, 169 parts, among them IC1 STMPS2141STR, IC10 74LCX245FT, IC11 74LCX245FT, IC12 LY68L6400SLIT, IC2 EP4CE6E22C8N, IC3 74LCX245FT, IC4 74LCX245FT, IC5 MP2233DJ, IC6 MP2233DJ, IC7 CH330N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

Commit message: Production
Parts:
- removed C55: 100nF 6.3V, GadgetFactory:0603
- removed U2: EPCS16, Altera_By_element14_Batch_1:SOIC127P600X175-8N
- added TP4, TP5: TPTP08R, testpad:TP08R
- moved R4 0.50 mm to (19.4, 44.0)
Connections:
- removed net ASDO: IC2.6, U2.5
- removed net DATA0: IC2.13, U2.2
- removed net DCLK: IC2.12, U2.6
- removed net NCSO: IC2.8, U2.1
- new net N$1: IC2.8, TP4.TP
- new net N$55: IC2.144, TP5.TP
- net +3V3: no longer C55.1, IC2.94, U2.3, U2.7, U2.8
- net ESP_MISO: now also IC2.6; no longer IC2.2
- net ESP_MOSI: now also IC2.13; no longer IC2.144
- net ESP_SCK: now also IC2.12
- net GND: now also IC2.94; no longer C55.2, U2.4
- net LED2: now also IC2.2; no longer U1.9
- net NSTATUS: now also U1.27
- net PULLUP_EN: now also U1.9; no longer U1.27
Routing:
- net NSTATUS: track 2.51 -> 45.6 mm, vias 1 -> 10
- net LED2: track 12.9 -> 31.3 mm, vias 1 -> 2
- net NCSO: track 16.2 -> 0.00 mm
- net DATA0: track 15.1 -> 0.00 mm, vias 2 -> 0
- net +3V3: track 488.0 -> 473.9 mm
- net ASDO: track 9.31 -> 0.00 mm, vias 2 -> 0
- net PULLUP_EN: track 21.9 -> 31.0 mm, vias 4 -> 6
- net DCLK: track 8.46 -> 0.00 mm
- net ESP_SCK: track 42.4 -> 50.5 mm, vias 3 -> 5
- net ESP_MOSI: track 43.2 -> 49.2 mm, vias 1 -> 3
- net GND: track 118.3 -> 115.6 mm, vias 196 -> 207
- net N$1: track 0.00 -> 2.65 mm
- net A2: track 9.82 -> 12.3 mm
- net ESP_NCS0: track 43.8 -> 45.6 mm
- net N$55: track 0.00 -> 1.33 mm
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
Commit message: Fix resistor value
Parts:
- RN7, RN8: value 330R -> 33R
Changed lines of the file:
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@@
 <layer number="14" name="Route14" color="1" fill="6" visible="no" active="no"/>
 <layer number="15" name="Route15" color="4" fill="6" visible="no" active="no"/>
-<layer number="16" name="Bottom" color="1" fill="1" visible="no" active="yes"/>
+<layer number="16" name="Bottom" color="1" fill="1" visible="yes" active="yes"/>
 <layer number="17" name="Pads" color="2" fill="1" visible="yes" active="yes"/>
 <layer number="18" name="Vias" color="2" fill="1" visible="yes" active="yes"/>
@@
 <layer number="20" name="Dimension" color="15" fill="1" visible="yes" active="yes"/>
 <layer number="21" name="tPlace" color="7" fill="1" visible="yes" active="yes"/>
-<layer number="22" name="bPlace" color="7" fill="1" visible="no" active="yes"/>
+<layer number="22" name="bPlace" color="7" fill="1" visible="yes" active="yes"/>
 <layer number="23" name="tOrigins" color="15" fill="1" visible="yes" active="yes"/>
-<layer number="24" name="bOrigins" color="15" fill="1" visible="no" active="yes"/>
+<layer number="24" name="bOrigins" color="15" fill="1" visible="yes" active="yes"/>
 <layer number="25" name="tNames" color="7" fill="1" visible="yes" active="yes"/>
-<layer number="26" name="bNames" color="7" fill="1" visible="no" active="yes"/>
+<layer number="26" name="bNames" color="7" fill="1" visible="yes" active="yes"/>
 <layer number="27" name="tValues" color="7" fill="1" visible="no" active="yes"/>
 <layer number="28" name="bValues" color="7" fill="1" visible="no" active="yes"/>
@@
 <layer number="43" name="vRestrict" color="2" fill="10" visible="no" active="yes"/>
 <layer number="44" name="Drills" color="7" fill="1" visible="no" active="yes"/>
-<layer number="45" name="Holes" color="7" fill="1" visible="no" active="yes"/>
+<layer number="45" name="Holes" color="7" fill="1" visible="yes" active="yes"/>
 <layer number="46" name="Milling" color="3" fill="1" visible="no" active="yes"/>
 <layer number="47" name="Measures" color="7" fill="1" visible="no" active="yes"/>
-<layer number="48" name="Document" color="7" fill="1" visible="no" active="yes"/>
+<layer number="48" name="Document" color="7" fill="1" visible="yes" active="yes"/>
 <layer number="49" name="Reference" color="7" fill="1" visible="no" active="yes"/>
 <layer number="50" name="dxf" color="7" fill="1" visible="no" active="no"/>
-<layer number="51" name="tDocu" color="7" fill="1" visible="no" active="yes"/>
-<layer number="52" name="bDocu" color="7" fill="1" visible="no" active="yes"/>
+<layer number="51" name="tDocu" color="7" fill="1" visible="yes" active="yes"/>
+<layer number="52" name="bDocu" color="7" fill="1" visible="yes" active="yes"/>
 <layer number="53" name="tGND_GNDA" color="7" fill="1" visible="no" active="no"/>
 <layer number="54" name="bGND_GNDA" color="7" fill="1" visible="no" active="no"/>
@@
 <attribute name="VALUE" x="51.4012" y="13.0072" size="1.016" layer="27" ratio="10" rot="R90"/>
 </element>
-<element name="RN7" library="resistor-dil" package="EXB28V" value="330R" x="44.945" y="10.355" smashed="yes">
+<element name="RN7" library="resistor-dil" package="EXB28V" value="33R" x="44.945" y="10.355" smashed="yes">
 <attribute name="OC_NEWARK" value="unknown" x="41.135" y="16.705" size="1.778" layer="27" display="off"/>
 <attribute name="MPN" value="" x="41.135" y="16.705" size="1.778" layer="27" display="off"/>
@@
 <attribute name="VALUE" x="43.9925" y="8.1325" size="1.27" layer="27"/>
 </element>
-<element name="RN8" library="resistor-dil" package="EXB28V" value="330R" x="47.785" y="10.355" smashed="yes">
+<element name="RN8" library="resistor-dil" package="EXB28V" value="33R" x="47.785" y="10.355" smashed="yes">
 <attribute name="OC_NEWARK" value="unknown" x="36.355" y="16.705" size="1.778" layer="27" display="off"/>
 <attribute name="MPN" value="" x="36.355" y="16.705" size="1.778" layer="27" display="off"/>
