File: pcb/interfacez_r2_1.sch (EAGLE design)
At the start: 169 parts, among them IC1 STMPS2141STR, IC10 74LCX245FT, IC11 74LCX245FT, IC12 LY68L6400SLIT, IC2 EP4CE6E22C8N, IC3 74LCX245FT, IC4 74LCX245FT, IC5 MP2233DJ, IC6 MP2233DJ, IC7 CH330N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

Commit message: Production
Parts:
- removed C55: 100nF 6.3V, GadgetFactory:C0603
- removed U2: EPCS16, Altera_By_element14_Batch_1:EPCS1SI8N
- added TP4, TP5: TPTP08R, testpad:TPTP08R
Connections:
- removed net ASDO: IC2.__IO_4/DATA/ADSO, U2.ASDI
- removed net DATA0: IC2.__DATA0, U2.DATA
- removed net DCLK: IC2.__DCLK, U2.DCLK
- removed net NCSO: IC2.__IO_6/FLASH_NCS/NCSO, U2.NCS
- new net N$1: IC2.__IO_6/FLASH_NCS/NCSO, TP4.TP
- new net N$55: IC2.__IO_84, TP5.TP
- net +3V3: no longer C55.1, IC2.__MSEL0, U2.VCC, U2.VCC_2, U2.VCC_3
- net ESP_MISO: now also IC2.__IO_4/DATA/ADSO; no longer IC2.__IO_2
- net ESP_MOSI: now also IC2.__DATA0; no longer IC2.__IO_84
- net ESP_SCK: now also IC2.__DCLK
- net GND: now also IC2.__MSEL0; no longer C55.2, U2.GND
- net LED2: now also IC2.__IO_2; no longer U1.IO33
- net NSTATUS: now also U1.IO16
- net PULLUP_EN: now also U1.IO33; no longer U1.IO16
Other:
- note added: "CHANGE TO PS!"
- note added: "DMC3400SDW-7"

Commit message: Fix resistor value
Parts:
- RN7, RN8: value 330R -> 33R
Changed lines of the file:
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@@
 <part name="RN6" library="resistor-dil" deviceset="4R-N" device="EXB28V" value="330R"/>
 <part name="IC4" library="GadgetFactory" deviceset="74*245" device="" value="74LCX245FT"/>
-<part name="RN7" library="resistor-dil" deviceset="4R-N" device="EXB28V" value="330R"/>
-<part name="RN8" library="resistor-dil" deviceset="4R-N" device="EXB28V" value="330R"/>
+<part name="RN7" library="resistor-dil" deviceset="4R-N" device="EXB28V" value="33R"/>
+<part name="RN8" library="resistor-dil" deviceset="4R-N" device="EXB28V" value="33R"/>
 <part name="R8" library="GadgetFactory" deviceset="R" device="0603" value="10K"/>
 <part name="R9" library="GadgetFactory" deviceset="R" device="0603" value="10K"/>

Commit message: Working
Other:
- note added: "IO2 NEEDS PULLDOWN FOR SERIAL PROG!"
- note added: "NEEDS 15K PULLDOWNS!"
Changed lines of the file:
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@@
 <text x="619.76" y="424.18" size="1.778" layer="91">CHANGE TO PS!</text>
 <text x="190.5" y="139.7" size="1.778" layer="91">DMC3400SDW-7</text>
+<text x="243.84" y="-58.42" size="1.778" layer="97">NEEDS 15K PULLDOWNS!</text>
+<text x="71.12" y="307.34" size="1.778" layer="97">IO2 NEEDS PULLDOWN FOR SERIAL PROG!</text>
 </plain>
 <instances>

Commit message: USB layer and cleanups
Other:
- note added: "+3 NOE for second ROM"
- note added: "Consider USB1T11A"
Changed lines of the file:
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@@
 <text x="243.84" y="-58.42" size="1.778" layer="97">NEEDS 15K PULLDOWNS!</text>
 <text x="71.12" y="307.34" size="1.778" layer="97">IO2 NEEDS PULLDOWN FOR SERIAL PROG!</text>
+<text x="83.82" y="208.28" size="1.778" layer="97">+3 NOE for second ROM</text>
+<text x="213.36" y="-78.74" size="1.778" layer="97">Consider USB1T11A</text>
 </plain>
 <instances>
