File: pcb/interfacez_r2_2.brd (EAGLE design)
At the start: 100 x 50 mm, 171 parts, among them IC1 STMPS2141STR, IC10 74LCX245FT, IC11 74LCX245FT, IC12 USB1T11AMTCX, IC2 EP4CE6E22C8N, IC3 74LCX245FT, IC4 74LCX245FT, IC5 MP2233DJ, IC6 MP2233DJ, IC7 CH330N, IC8 MIC5504-2.5YM5-TR, IC9 LY68L6400SLIT, Q1 BSS123, Q2 BSS123, Q3 CJ3439KDW, Q4 CJ3439KDW, Q5 BSS84, Q6 BSS123, U1 ESP-WROOM-32

Commit message: PCB 2.2 updates
Parts:
- removed CONN2: PIN-2X5, alvie:PIN-2X5
- added J1: AMPHENOL_ICC_-_FCI_20021121-00010C4LFAMPHENOL_ICC_-_FCI_200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, 20021121-00010C4LF:AMPHENOL_ICC_-_FCI_20021121-00010C4LF_0
- moved R8 13.1 mm to (32.0, 38.1), flipped to the bottom, turned to 90 degrees
- moved R9 11.0 mm to (33.4, 38.1), flipped to the bottom, turned to 90 degrees
- moved R10 7.42 mm to (29.0, 36.1), turned to 0 degrees
- moved U$7 5.75 mm to (49.5, 48.4)
- moved TP3 3.62 mm to (25.9, 35.9)
- moved C49 2.20 mm to (76.2, 27.1), flipped to the top
- moved TP4 1.09 mm to (38.6, 38.6)
- moved R6 0.69 mm to (39.6, 37.5), turned to 270 degrees
Connections:
- new net N$66: J1.7
- new net N$70: J1.6
- new net N$71: J1.8
- net +3V3: now also J1.4; no longer CONN2.4
- net GND: now also J1.10, J1.2; no longer CONN2.10, CONN2.2
- net RAMD0: now also IC2.83; no longer IC2.99
- net RAMD1: now also IC2.87; no longer IC2.98
- net RAMD2: now also IC2.86; no longer IC2.87
- net RAMD3: now also IC2.85; no longer IC2.100
- net RAMNCS: now also IC2.98; no longer IC2.101
- net TCK: now also J1.1; no longer CONN2.1
- net TDI: now also J1.9; no longer CONN2.9
- net TDO: now also J1.3; no longer CONN2.3
- net TMS: now also J1.5; no longer CONN2.5
Routing:
- net TDO: track 32.8 -> 12.2 mm
- net TMS: track 29.3 -> 10.5 mm
- net TDI: track 14.6 -> 4.86 mm, vias 3 -> 0
- net TCK: track 24.1 -> 14.6 mm, vias 1 -> 3
- net EXT7: track 16.1 -> 10.4 mm
- net EXT4: track 11.4 -> 5.70 mm
- net EXT6: track 16.5 -> 10.8 mm
- net RAMD1: track 15.0 -> 9.72 mm
- net EXT5: track 15.3 -> 10.0 mm
- net EXT3: track 9.56 -> 4.70 mm
- net NSTATUS: track 44.7 -> 48.2 mm, vias 10 -> 5
- net RAMD0: track 21.9 -> 18.6 mm
- net RAMCLK: track 21.4 -> 18.9 mm, vias 2 -> 0
- net RAMNCS: track 15.4 -> 13.0 mm, vias 2 -> 0
- net EXT2: track 7.81 -> 5.43 mm
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
Commit message: New board layout
Parts:
- removed SJ1: (no value), jumper:SJ_2
- removed TP5: TPTP08R, testpad:TP08R
- removed U$2: PIN-1X10, alvie:PIN-1X10
- added C54, C61, C63: 100nF, GadgetFactory:0603
- added C55, C62: 47uF, GadgetFactory:1206
- added IC13: NC7WZ16P6X, GadgetFactory:SC70-6
- added R58: 520R, GadgetFactory:0603
- added R59, R60: 270R, GadgetFactory:0603
- added R61, R64: 220R, GadgetFactory:0603
- added R62, R65: 100R, GadgetFactory:0603
- added R63, R66: 1K8, GadgetFactory:0603
- added R67, R68: 0R/DNP, GadgetFactory:0603
- added U$5, U$8: INTERFACEZ_EDGEDAUGHTER, alvie:INTERFACEZ_EXPANSION_DAUGHTERCARD
- added U$9: PJ328-A0, alvie:PJ328A0
- moved R50 86.8 mm to (10.7, 22.5), flipped to the top, turned to 270 degrees
- moved R47 82.3 mm to (8.00, 17.1), flipped to the top, turned to 0 degrees
- moved R52 82.3 mm to (8.00, 11.9), flipped to the top, turned to 0 degrees
- moved R46 82.2 mm to (8.05, 14.5), flipped to the top, turned to 0 degrees
- moved R51 82.2 mm to (8.05, 9.45), flipped to the top, turned to 0 degrees
- moved R53 82.2 mm to (8.05, 4.35), flipped to the top, turned to 0 degrees
- moved R54 82.2 mm to (8.05, 6.90), flipped to the top, turned to 0 degrees
- moved R56 82.2 mm to (8.05, 1.85), flipped to the top, turned to 0 degrees
- moved R49 81.8 mm to (12.2, 22.5), flipped to the top
- moved R55 79.1 mm to (11.2, 2.80), flipped to the top, turned to 0 degrees
- moved R48 77.5 mm to (13.7, 22.5), flipped to the top
- moved X1 76.0 mm to (19.5, 17.5)
- moved USB2 49.0 mm to (76.5, 91.0)
- moved C50 46.2 mm to (65.6, 91.2), flipped to the top, turned to 180 degrees
- moved R45 45.0 mm to (66.9, 87.6), flipped to the top, turned to 270 degrees
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Connections:
- removed net N$66: J1.7
- removed net N$70: J1.6
- removed net N$71: J1.8
- removed net SPEED: IC12.9, IC2.112
- removed net VREG: C31.2, C32.2, C33.2, C34.2, IC5.2, IC6.2, SJ1.2
- new net AUDIO_L: IC13.3, R68.1, U$8.A6
- new net AUDIO_R: IC13.1, R67.1, U$8.A5
- new net BLUE2: R60.1, U$8.A9
- new net BUF_L: IC13.6, R64.2, R67.2
- new net BUF_R: IC13.4, R61.2, R68.2
- new net EXT10: IC2.115, U$5.A8
- new net EXT11: IC2.114, U$5.A9
- new net EXT12: IC2.142, U$5.A5
- new net EXT13: IC2.144, U$5.A4
- new net EXT8: IC2.120, U$5.A6
- new net EXT9: IC2.119, U$5.A7
- new net GREEN2: R59.1, U$8.A7
- new net LL: C62.2, R66.1, U$9.2
- new net LR: C55.2, R63.1, U$9.3
- new net N$67: C61.2, C62.1, R64.1, R65.1
- new net N$68: C54.2, C55.1, R61.1, R62.1
- new net RED2: R58.1, U$8.A8
- new net USB_SPEED: IC12.9, IC2.106
- net +3V3: now also C63.2, IC13.5, U$5.B1, U$8.B1; no longer U$2.1
- net +5V: now also U$5.A1; no longer SJ1.1
- net +9V: now also C31.2, C32.2, C33.2, C34.2, IC5.2, IC6.2; no longer SJ1.3
- net BLUE: now also R60.2
- net BLUE0: now also U$8.A10; no longer U$2.10
- net BLUE1: now also U$8.B10; no longer U$2.9
- net EXT0: now also U$5.B4
- net EXT1: now also U$5.B5
- net EXT2: now also U$5.B6
- net EXT3: now also U$5.B7
- net EXT4: now also U$5.B8
- net EXT5: now also U$5.B9
- net EXT6: now also U$5.B10
- net EXT7: now also U$5.A10
- net GND: now also C54.1, C61.1, C63.1, IC13.2, R62.2, R63.2, R65.2, R66.2, U$5.A2, U$5.B2, U$8.A2, U$8.B2, U$9.1; no longer U$2.2
- net GREEN: now also R59.2
- net GREEN0: now also U$8.B9; no longer U$2.8
- net GREEN1: now also U$8.B8; no longer U$2.7
- net HSYNC: now also U$8.B4; no longer U$2.3
- net N$55: now also U$8.A1; no longer IC2.144, TP5.TP
- net RCV: now also IC2.103; no longer IC2.106
- net RED: now also R58.2
- net RED0: now also U$8.B7; no longer U$2.6
- net RED1: now also U$8.B6; no longer U$2.5
- net USB_FLT: now also IC2.112; no longer IC2.115
- net USB_MODE: now also IC2.105; no longer IC2.111
- net USB_OE: now also IC2.104; no longer IC2.110
- net USB_PWREN: now also IC2.113; no longer IC2.119
- net USB_SUSPEND: now also IC2.99; no longer IC2.103
- net VM: now also IC2.100; no longer IC2.104
- net VMO: now also IC2.111; no longer IC2.114
- net VP: now also IC2.101; no longer IC2.105
- net VPO: now also IC2.110; no longer IC2.113
- net VSYNC: now also U$8.B5; no longer U$2.4
Routing:
- net GND: track 112.0 -> 163.4 mm, vias 206 -> 231
- net +3V3: track 484.5 -> 529.0 mm, vias 69 -> 70
- net SPEED: track 25.4 -> 0.00 mm
- net +9V: track 6.01 -> 29.8 mm, vias 0 -> 4
- net VREG: track 23.1 -> 0.00 mm, vias 2 -> 0
- net +5V: track 172.7 -> 195.4 mm, vias 19 -> 23
- net AUDIO_L: track 0.00 -> 22.6 mm, vias 0 -> 1
- net GREEN: track 14.7 -> 36.6 mm, vias 1 -> 3
- net AUDIO_R: track 0.00 -> 20.1 mm, vias 0 -> 1
- net EXT8: track 0.00 -> 18.7 mm, vias 0 -> 1
- net LR: track 0.00 -> 18.5 mm
- net USB_SPEED: track 0.00 -> 17.3 mm
- net EXT9: track 0.00 -> 17.2 mm, vias 0 -> 1
- net BLUE: track 17.8 -> 34.8 mm, vias 2 -> 3
- net EXT10: track 0.00 -> 15.7 mm, vias 0 -> 1
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- added copper zone on layer 1, net +9V
- removed copper zone on layer 1, net VREG
Other:
- board size 100 x 50 mm -> 86 x 100 mm
- board text added: "AUDIO"
- board text added: "E0"
- board text added: "E1"
- board text added: "E10"
- board text added: "E11"
- board text added: "E12"
- board text added: "E13"
- board text added: "E2"
- board text added: "E3"
- board text added: "E4"
- board text added: "E5"
- board text added: "E6"
- board text added: "E7"
- board text added: "E8"
- board text added: "E9"
- board text added: "OUT"
- board text added: "Open Source Hardware: CC-BY-SA"
- board text added: "Rev. 2.2"
- board text removed: "+9V"
- board text removed: "Rev. 2"
- board text removed: "ZX Spectrum Interface Z"

Commit message: r2.2 updates
Parts:
- added JP1: (no value), SparkFun-Connectors:2X10
- added U$2: INTERFACEZ_EDGEDAUGHTER, alvie:INTERFACEZ_EXPANSION_DAUGHTERCARD
- R51, R53, R55: value 520R -> 1K24
- R52, R54, R56: value 270R -> 619R
- R58: value 520R -> 309R
- R59, R60: value 270R -> 309R
Connections:
- new net N$61: U$2.A1
- net +3V3: now also U$2.B1
- net AUDIO_L: now also U$2.A6
- net AUDIO_R: now also U$2.A5
- net BLUE0: now also U$2.A10
- net BLUE1: now also U$2.B10
- net BLUE2: now also U$2.A9
- net GND: now also U$2.A2, U$2.B2
- net GREEN0: now also U$2.B9
- net GREEN1: now also U$2.B8
- net GREEN2: now also U$2.A7
- net HSYNC: now also U$2.B4
- net RED0: now also U$2.B7
- net RED1: now also U$2.B6
- net RED2: now also U$2.A8
- net VSYNC: now also U$2.B5

Commit message: Rev 2.2 for board
Parts:
- added C100, C101, C93, C94, C95: 100nF, GadgetFactory:0603
- added C64, C66: 100nF 6.3V, GadgetFactory:0603
- added C65: 47uF 6.3V TANT, alvie:TANT_CASE_A
- added C96: 2.2uF, GadgetFactory:0805
- added C97: 1uF, GadgetFactory:0603
- added C98: 1nF, GadgetFactory:0603
- added C99: 100nF/DNP, GadgetFactory:0603
- added IC14: LAN8720A, sigedi-footprints:QFN24_4MM_X_4MM
- added L8: 600R, GadgetFactory:0805
- added R69, R70, R71, R79, R80: 2K2, GadgetFactory:0603
- added R78: 10K, GadgetFactory:0603
- added R81: 0R, GadgetFactory:0603
- added R82: 12K1, GadgetFactory:0603
- added R83, R84, R85, R86: 49R9, GadgetFactory:0603
- added R87, R88: 330R, GadgetFactory:0603
- added T1: Hanrun HR917550A, alvie:HR13550A
- added U$10: INTERFACEZ_EDGEDAUGHTER, alvie:INTERFACEZ_EXPANSION_DAUGHTERCARD
- added U$11, U$6: PMS150C-U06, alvie:SOT23-6
- added U$12, U$13: (no value), interfacez:LOGO-20
- added U$14: (no value), interfacez:LOGO-23-2.65
- added U$15: PIN-2X5-1.27MM, alvie:PIN-2X5-1.27
- added U$16: PIN-2X5, alvie:PIN-2X5
- moved C51 3.12 mm to (11.3, 80.8), flipped to the top, turned to 0 degrees
- moved JP1 0.25 mm to (47.0, 13.0), turned to 270 degrees
Connections:
- new net CLKIN: R81.1, U$10.B4
- new net ETHID: R71.1, U$10.A4, U$11.3
- new net ETH_CLK: IC14.5, R81.2
- new net ETH_CRS_DV: IC14.11, U$10.B7
- new net ETH_MDC: IC14.13, R79.1, U$10.A8
- new net ETH_MDIO: IC14.12, R80.1, U$10.A7
- new net ETH_NRST: IC14.15, R78.1, U$10.A9
- new net ETH_REF_CLK: IC14.14, U$10.B8
- new net ETH_RXD0: IC14.8, U$10.B6
- new net ETH_RXD1: IC14.7, U$10.B5
- new net ETH_RXERR: IC14.10, U$10.A6
- new net ETH_TXD0: IC14.17, U$10.A10
- new net ETH_TXD1: IC14.18, U$10.B10
- new net ETH_TX_EN: IC14.16, U$10.B9
- new net EXTID: JP1.8, R70.1, U$2.A4
- new net N$64: C101.1, T1.5
- new net N$65: C100.1, T1.4
- new net N$66: JP1.7, U$2.B4
- new net N$69: JP1.9, U$2.B5
- new net N$70: JP1.11, U$2.B6
- new net N$71: JP1.13, U$2.B7
- new net N$72: JP1.15, U$2.B8
- new net N$73: JP1.17, U$2.B9
- new net N$74: JP1.19, U$2.B10
- new net N$75: C99.2, L8.2, R83.2, R84.2, R85.2, R86.2
- new net N$76: R87.2, T1.11
- new net N$77: JP1.10, U$2.A5
- new net N$78: JP1.12, U$2.A6
- new net N$79: JP1.14, U$2.A7
- new net N$80: JP1.16, U$2.A8
- new net N$81: JP1.18, U$2.A9
- new net N$82: JP1.20, U$2.A10
- new net N$83: R88.2, T1.10
- new net N$84: IC14.24, R82.2
- new net N$85: C97.2, C98.2, IC14.6
- new net N$86: U$15.1, U$16.1
- new net N$87: U$15.3, U$16.3
- new net N$88: U$15.5, U$16.5
- new net N$89: U$15.7, U$16.7
- new net N$90: U$15.9, U$16.9
- new net N$91: U$15.2, U$16.2
- new net N$92: U$15.4, U$16.4
- new net N$93: U$15.6, U$16.6
- new net N$94: U$15.8, U$16.8
- new net N$95: U$15.10, U$16.10
- new net NC: U$10.A1
- new net PHY_LED0: IC14.3, T1.12
- new net PHY_LED1: IC14.2, T1.9
- new net RXM: IC14.20, R84.1, T1.2
- new net RXP: IC14.21, R83.1, T1.1
- new net TXM: IC14.22, R86.1, T1.6
- new net TXP: IC14.23, R85.1, T1.3
- new net VGAID: R69.1, U$6.3, U$8.A4
- net +3V3: now also C64.2, C65.PLUS, C66.2, C93.2, C94.2, C95.2, C96.2, IC14.1, IC14.19, IC14.9, JP1.1, L8.1, R69.2, R70.2, R71.2, R78.2, R79.2, R80.2, U$10.B1, U$11.5, U$6.5
- net AUDIO_L: no longer U$2.A6
- net AUDIO_R: no longer U$2.A5
- net BLUE0: no longer U$2.A10
- net BLUE1: no longer U$2.B10
- net BLUE2: no longer U$2.A9
- net GND: now also C100.2, C101.2, C64.1, C65.MINUS, C66.1, C93.1, C94.1, C95.1, C96.1, C97.1, C98.1, C99.1, IC14.P, JP1.3, JP1.4, R82.1, R87.1, R88.1, U$10.A2, U$10.B2, U$11.2, U$6.2
- net GREEN0: no longer U$2.B9
- net GREEN1: no longer U$2.B8
- net GREEN2: no longer U$2.A7
- net HSYNC: no longer U$2.B4
- net N$61: now also JP1.2
- net PE: now also T1.8, T1.Z1, T1.Z2
- net RED0: no longer U$2.B7
- net RED1: no longer U$2.B6
- net RED2: no longer U$2.A8
- net VSYNC: no longer U$2.B5
Routing:
- net +3V3: track 529.0 -> 704.3 mm, vias 70 -> 79
- net PE: track 19.6 -> 107.3 mm
- net TXP: track 0.00 -> 48.2 mm
- net TXM: track 0.00 -> 46.5 mm
- net GND: track 163.4 -> 207.4 mm, vias 231 -> 281
- net RXM: track 0.00 -> 41.1 mm, vias 0 -> 2
- net RXP: track 0.00 -> 39.7 mm, vias 0 -> 2
- net PHY_LED0: track 0.00 -> 33.7 mm, vias 0 -> 4
- net VGAID: track 0.00 -> 33.3 mm, vias 0 -> 3
- net N$88: track 0.00 -> 30.3 mm, vias 0 -> 2
- net N$89: track 0.00 -> 25.0 mm, vias 0 -> 2
- net ETH_NRST: track 0.00 -> 22.3 mm, vias 0 -> 3
- net N$87: track 0.00 -> 22.2 mm, vias 0 -> 2
- net ETH_TXD1: track 0.00 -> 19.7 mm
- net ETH_MDC: track 0.00 -> 19.6 mm, vias 0 -> 3
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Other:
- board text added: "+3V3"
- board text added: "E13/ DET"
- board text added: "Ethernet Adaptor"
- board text added: "VGA/Audio"
- board text removed: "AUDIO"
- board text removed: "OUT"

Commit message: Fix signal naming
Connections:
- net EXT10: now also IC2.119, U$5.A7; no longer IC2.115, U$5.A8
- net EXT11: now also IC2.120, U$5.A6; no longer IC2.114, U$5.A9
- net EXT8: now also IC2.114, U$5.A9; no longer IC2.120, U$5.A6
- net EXT9: now also IC2.115, U$5.A8; no longer IC2.119, U$5.A7
Routing:
- net EXT8: track 18.7 -> 13.9 mm
- net EXT11: track 13.9 -> 18.7 mm
- net EXT9: track 17.2 -> 15.7 mm
- net EXT10: track 15.7 -> 17.2 mm
Changed lines of the file:
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@@
 <grid distance="0.5" unitdist="mm" unit="mm" style="lines" multiple="1" display="yes" altdistance="0.05" altunitdist="mm" altunit="mm"/>
 <layers>
-<layer number="1" name="Top" color="4" fill="1" visible="no" active="yes"/>
+<layer number="1" name="Top" color="4" fill="1" visible="yes" active="yes"/>
 <layer number="2" name="Route2" color="1" fill="3" visible="no" active="yes"/>
 <layer number="3" name="Route3" color="4" fill="3" visible="no" active="no"/>
@@
 <layer number="19" name="Unrouted" color="6" fill="1" visible="no" active="yes"/>
 <layer number="20" name="Dimension" color="15" fill="1" visible="yes" active="yes"/>
-<layer number="21" name="tPlace" color="7" fill="1" visible="no" active="yes"/>
+<layer number="21" name="tPlace" color="7" fill="1" visible="yes" active="yes"/>
 <layer number="22" name="bPlace" color="7" fill="1" visible="yes" active="yes"/>
-<layer number="23" name="tOrigins" color="15" fill="1" visible="no" active="yes"/>
+<layer number="23" name="tOrigins" color="15" fill="1" visible="yes" active="yes"/>
 <layer number="24" name="bOrigins" color="15" fill="1" visible="yes" active="yes"/>
-<layer number="25" name="tNames" color="7" fill="1" visible="no" active="yes"/>
+<layer number="25" name="tNames" color="7" fill="1" visible="yes" active="yes"/>
 <layer number="26" name="bNames" color="7" fill="1" visible="yes" active="yes"/>
 <layer number="27" name="tValues" color="7" fill="1" visible="no" active="yes"/>
@@
 <wire x1="10.15" y1="76.7" x2="10.35" y2="76.9" width="0.1524" layer="1"/>
 </signal>
-<signal name="EXT8">
+<signal name="EXT11">
 <contactref element="IC2" pad="120"/>
 <contactref element="U$5" pad="A6"/>
@@
 <wire x1="45" y1="94.73" x2="45.02" y2="96.75" width="0.1524" layer="16"/>
 </signal>
-<signal name="EXT9">
+<signal name="EXT10">
 <contactref element="IC2" pad="119"/>
 <contactref element="U$5" pad="A7"/>
@@
 <wire x1="47.6" y1="94.71" x2="47.56" y2="96.75" width="0.1524" layer="16"/>
 </signal>
-<signal name="EXT10">
+<signal name="EXT9">
 <contactref element="IC2" pad="115"/>
 <contactref element="U$5" pad="A8"/>
@@
 <wire x1="50.1" y1="92.05" x2="50.1" y2="96.75" width="0.1524" layer="16"/>
 </signal>
-<signal name="EXT11">
+<signal name="EXT8">
 <contactref element="IC2" pad="114"/>
 <contactref element="U$5" pad="A9"/>
