File: pcb/interfacez_r2_2.sch (EAGLE design)
At the start: 171 parts, among them IC1 STMPS2141STR, IC10 74LCX245FT, IC11 74LCX245FT, IC12 USB1T11AMTCX, IC2 EP4CE6E22C8N, IC3 74LCX245FT, IC4 74LCX245FT, IC5 MP2233DJ, IC6 MP2233DJ, IC7 CH330N, IC8 MIC5504-2.5YM5-TR, IC9 LY68L6400SLIT, Q1 BSS123, Q2 BSS123, Q3 CJ3439KDW, Q4 CJ3439KDW, Q5 BSS84, Q6 BSS123, U1 ESP-WROOM-32

Commit message: PCB 2.2 updates
Parts:
- removed CONN2: PIN-2X5, alvie:PIN-2X5
- added J1: AMPHENOL_ICC_-_FCI_20021121-00010C4LFAMPHENOL_ICC_-_FCI_200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, 20021121-00010C4LF:AMPHENOL_ICC_-_FCI_20021121-00010C4LFAMPHENOL_ICC_-_FCI_20021121-00010C4LF_0_0
Connections:
- new net N$66: J1A.7
- new net N$70: J1B.6
- new net N$71: J1B.8
- net +3V3: now also J1B.4; no longer CONN2.4
- net GND: now also J1B.10, J1B.2; no longer CONN2.10, CONN2.2
- net RAMD0: now also IC2.__IO_47; no longer IC2.__IO_53
- net RAMD1: now also IC2.__IO_51; no longer IC2.__IO_52
- net RAMD2: now also IC2.__IO_50; no longer IC2.__IO_51
- net RAMD3: now also IC2.__IO_49; no longer IC2.__IO_54
- net RAMNCS: now also IC2.__IO_52; no longer IC2.__IO_55
- net TCK: now also J1A.1; no longer CONN2.1
- net TDI: now also J1A.9; no longer CONN2.9
- net TDO: now also J1A.3; no longer CONN2.3
- net TMS: now also J1A.5; no longer CONN2.5
Changed lines of the file:
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@@
 <part name="SD1" library="alvie" deviceset="1040310811" device=""/>
 <part name="GND120" library="supply1" deviceset="GND" device=""/>
-<part name="CONN2" library="alvie" deviceset="PIN-2X5" device=""/>
 <part name="GND45" library="supply1" deviceset="GND" device=""/>
 <part name="R1" library="GadgetFactory" deviceset="R" device="0603" value="10K"/>
@@
 <part name="+3V1" library="supply1" deviceset="+3V3" device=""/>
 <part name="C51" library="GadgetFactory" deviceset="C" device="0603" value="100nF 6.3V"/>
+<part name="J1" library="20021121-00010C4LF" deviceset="AMPHENOL_ICC_-_FCI_20021121-00010C4LF" device="AMPHENOL_ICC_-_FCI_20021121-00010C4LF_0_0"/>
 </parts>
 <sheets>
@@
 <instance part="SD1" gate="G$1" x="101.6" y="416.56"/>
 <instance part="GND120" gate="1" x="86.36" y="398.78" rot="MR0"/>
-<instance part="CONN2" gate="G$1" x="726.44" y="317.5" rot="MR180"/>
 <instance part="GND45" gate="1" x="751.84" y="322.58" rot="R90"/>
 <instance part="R1" gate="A" x="7.62" y="431.8" rot="R270"/>
@@
 <instance part="+3V1" gate="G$1" x="734.06" y="383.54"/>
 <instance part="C51" gate="A" x="734.06" y="370.84" rot="R90"/>
+<instance part="J1" gate="A" x="607.06" y="327.66"/>
+<instance part="J1" gate="B" x="645.16" y="327.66"/>
 </instances>
 <busses>
@@
 </segment>
 <segment>
-<pinref part="CONN2" gate="G$1" pin="2"/>
 <wire x1="736.6" y1="312.42" x2="739.14" y2="312.42" width="0.1524" layer="91"/>
 <wire x1="739.14" y1="312.42" x2="739.14" y2="304.8" width="0.1524" layer="91"/>
@@
 </segment>
 <segment>
-<pinref part="CONN2" gate="G$1" pin="10"/>
 <wire x1="736.6" y1="322.58" x2="749.3" y2="322.58" width="0.1524" layer="91"/>
 <pinref part="GND45" gate="1" pin="GND"/>
@@
 <junction x="734.06" y="363.22"/>
 </segment>
+<segment>
+<pinref part="J1" gate="B" pin="10"/>
+<wire x1="675.64" y1="297.18" x2="660.4" y2="297.18" width="0.1524" layer="91"/>
+<label x="668.02" y="297.18" size="1.778" layer="95"/>
+</segment>
+<segment>
+<pinref part="J1" gate="B" pin="2"/>
+<wire x1="660.4" y1="317.5" x2="675.64" y2="317.5" width="0.1524" layer="91"/>
+<label x="668.02" y="317.5" size="1.778" layer="95"/>
+</segment>
 </net>
 <net name="N$149" class="0">
@@
 <wire x1="736.6" y1="314.96" x2="749.3" y2="314.96" width="0.1524" layer="91"/>
 <label x="739.14" y="314.96" size="1.778" layer="95"/>
-<pinref part="CONN2" gate="G$1" pin="4"/>
 </segment>
 <segment>
@@
 <junction x="734.06" y="378.46"/>
 </segment>
+<segment>
+<pinref part="J1" gate="B" pin="4"/>
+<wire x1="675.64" y1="312.42" x2="660.4" y2="312.42" width="0.1524" layer="91"/>
+<label x="668.02" y="312.42" size="1.778" layer="95"/>
+</segment>
 </net>
 <net name="ESP_TX" class="0">
@@
 <segment>
 <label x="706.12" y="322.58" size="1.778" layer="95"/>
-<pinref part="CONN2" gate="G$1" pin="9"/>
 <wire x1="716.28" y1="322.58" x2="706.12" y2="322.58" width="0.1524" layer="91"/>
 </segment>
+<segment>
+<pinref part="J1" gate="A" pin="9"/>
+<wire x1="635" y1="297.18" x2="622.3" y2="297.18" width="0.1524" layer="91"/>
+<label x="627.38" y="297.18" size="1.778" layer="95"/>
+</segment>
 </net>
 <net name="TCK" class="0">
@@
 <wire x1="716.28" y1="312.42" x2="703.58" y2="312.42" width="0.1524" layer="91"/>
 <wire x1="703.58" y1="312.42" x2="703.58" y2="309.88" width="0.1524" layer="91"/>
-<pinref part="CONN2" gate="G$1" pin="1"/>
+</segment>
+<segment>
+<pinref part="J1" gate="A" pin="1"/>
+<wire x1="622.3" y1="317.5" x2="635" y2="317.5" width="0.1524" layer="91"/>
+<label x="627.38" y="317.5" size="1.778" layer="95"/>
 </segment>
 </net>
@@
 <wire x1="716.28" y1="317.5" x2="698.5" y2="317.5" width="0.1524" layer="91"/>
 <wire x1="698.5" y1="317.5" x2="698.5" y2="320.04" width="0.1524" layer="91"/>
-<pinref part="CONN2" gate="G$1" pin="5"/>
+</segment>
+<segment>
+<pinref part="J1" gate="A" pin="5"/>
+<wire x1="635" y1="307.34" x2="622.3" y2="307.34" width="0.1524" layer="91"/>
+<label x="627.38" y="307.34" size="1.778" layer="95"/>
 </segment>
 </net>
@@
 <wire x1="716.28" y1="314.96" x2="693.42" y2="314.96" width="0.1524" layer="91"/>
 <wire x1="693.42" y1="314.96" x2="693.42" y2="320.04" width="0.1524" layer="91"/>
-<pinref part="CONN2" gate="G$1" pin="3"/>
+</segment>
+<segment>
+<pinref part="J1" gate="A" pin="3"/>
+<wire x1="632.46" y1="312.42" x2="622.3" y2="312.42" width="0.1524" layer="91"/>
+<label x="627.38" y="312.42" size="1.778" layer="95"/>
 </segment>
 </net>
@@
 </segment>
 <segment>
-<pinref part="IC2" gate="G$1" pin="__IO_55"/>
-<wire x1="584.2" y1="436.88" x2="599.44" y2="436.88" width="0.1524" layer="91"/>
-<label x="586.74" y="436.88" size="1.778" layer="95"/>
+<pinref part="IC2" gate="G$1" pin="__IO_52"/>
+<wire x1="584.2" y1="429.26" x2="596.9" y2="429.26" width="0.1524" layer="91"/>
+<label x="586.74" y="429.26" size="1.778" layer="95"/>
 </segment>
 </net>
@@
 </segment>
 <segment>
-<pinref part="IC2" gate="G$1" pin="__IO_53"/>
-<wire x1="584.2" y1="431.8" x2="596.9" y2="431.8" width="0.1524" layer="91"/>
-<label x="586.74" y="431.8" size="1.778" layer="95"/>
+<pinref part="IC2" gate="G$1" pin="__IO_47"/>
+<wire x1="584.2" y1="391.16" x2="594.36" y2="391.16" width="0.1524" layer="91"/>
+<label x="586.74" y="391.16" size="1.778" layer="95"/>
 </segment>
 </net>
@@
 </segment>
 <segment>
-<pinref part="IC2" gate="G$1" pin="__IO_52"/>
-<wire x1="584.2" y1="429.26" x2="596.9" y2="429.26" width="0.1524" layer="91"/>
-<label x="586.74" y="429.26" size="1.778" layer="95"/>
+<pinref part="IC2" gate="G$1" pin="__IO_51"/>
+<wire x1="584.2" y1="401.32" x2="594.36" y2="401.32" width="0.1524" layer="91"/>
+<label x="586.74" y="401.32" size="1.778" layer="95"/>
 </segment>
 </net>
@@
 </segment>
 <segment>
-<pinref part="IC2" gate="G$1" pin="__IO_51"/>
-<wire x1="584.2" y1="401.32" x2="594.36" y2="401.32" width="0.1524" layer="91"/>
-<label x="586.74" y="401.32" size="1.778" layer="95"/>
+<pinref part="IC2" gate="G$1" pin="__IO_50"/>
+<wire x1="584.2" y1="398.78" x2="594.36" y2="398.78" width="0.1524" layer="91"/>
+<label x="586.74" y="398.78" size="1.778" layer="95"/>
 </segment>
 </net>
@@
 </segment>
 <segment>
-<pinref part="IC2" gate="G$1" pin="__IO_54"/>
-<wire x1="584.2" y1="434.34" x2="596.9" y2="434.34" width="0.1524" layer="91"/>
-<label x="586.74" y="434.34" size="1.778" layer="95"/>
+<pinref part="IC2" gate="G$1" pin="__IO_49"/>
+<wire x1="584.2" y1="396.24" x2="594.36" y2="396.24" width="0.1524" layer="91"/>
+<label x="586.74" y="396.24" size="1.778" layer="95"/>
 </segment>
 </net>
@@
 </segment>
 </net>
+<net name="N$66" class="0">
+<segment>
+<pinref part="J1" gate="A" pin="7"/>
+<wire x1="632.46" y1="302.26" x2="622.3" y2="302.26" width="0.1524" layer="91"/>
+</segment>
+</net>
+<net name="N$70" class="0">
+<segment>
+<pinref part="J1" gate="B" pin="6"/>
+<wire x1="675.64" y1="307.34" x2="660.4" y2="307.34" width="0.1524" layer="91"/>
+</segment>
+</net>
+<net name="N$71" class="0">
+<segment>
+<pinref part="J1" gate="B" pin="8"/>
+<wire x1="660.4" y1="302.26" x2="675.64" y2="302.26" width="0.1524" layer="91"/>
+</segment>
+</net>

Commit message: New board layout
Parts:
- removed SJ1: (no value), jumper:SJ2W
- removed TP5: TPTP08R, testpad:TPTP08R
- removed U$2: PIN-1X10, alvie:PIN-1X10
- added C54, C61, C63: 100nF, GadgetFactory:C0603
- added C55, C62: 47uF, GadgetFactory:C1206
- added IC13: NC7WZ16P6X, GadgetFactory:NC7WZ07P6X
- added R58: 520R, GadgetFactory:R0603
- added R59, R60: 270R, GadgetFactory:R0603
- added R61, R64: 220R, GadgetFactory:R0603
- added R62, R65: 100R, GadgetFactory:R0603
- added R63, R66: 1K8, GadgetFactory:R0603
- added R67, R68: 0R/DNP, GadgetFactory:R0603
- added U$5, U$8: INTERFACEZ_EDGEDAUGHTER, alvie:INTERFACEZ_EDGEDAUGHTER
- added U$9: PJ328-A0, alvie:PJ328-A0
Connections:
- removed net N$66: J1A.7
- removed net N$70: J1B.6
- removed net N$71: J1B.8
- removed net SPEED: IC12.SPEED, IC2.__IO_62
- removed net VREG: C31.2, C32.2, C33.2, C34.2, IC5.IN, IC6.IN, SJ1.2
- new net AUDIO_L: IC13GATE2.I, R68A.1, U$8.E11
- new net AUDIO_R: IC13GATE1.I, R67A.1, U$8.E12
- new net BLUE2: R60A.1, U$8.E8
- new net BUF_L: IC13GATE1.O, R64A.2, R67A.2
- new net BUF_R: IC13GATE2.O, R61A.2, R68A.2
- new net EXT10: IC2.__IO_65, U$5.E9
- new net EXT11: IC2.__IO_64, U$5.E8
- new net EXT12: IC2.__IO_82, U$5.E12
- new net EXT13: IC2.__IO_84, U$5.E13
- new net EXT8: IC2.__IO_67, U$5.E11
- new net EXT9: IC2.__IO_66, U$5.E10
- new net GREEN2: R59A.1, U$8.E10
- new net LL: C62.2, R66A.1, U$9.TIP
- new net LR: C55.2, R63A.1, U$9.RING
- new net N$67: C61.2, C62.1, R64A.1, R65A.1
- new net N$68: C54.2, C55.1, R61A.1, R62A.1
- new net RED2: R58A.1, U$8.E9
- new net USB_SPEED: IC12.SPEED, IC2.__IO_59
- net +3V3: now also C63.2, IC13G$3.VCC, U$5.+3V3, U$8.+3V3; no longer U$2.1
- net +5V: now also U$5.+5V; no longer SJ1.1
- net +9V: now also C31.2, C32.2, C33.2, C34.2, IC5.IN, IC6.IN; no longer SJ1.3
- net BLUE: now also R60A.2
- net BLUE0: now also U$8.E7; no longer U$2.10
- net BLUE1: now also U$8.E6; no longer U$2.9
- net EXT0: now also U$5.E0
- net EXT1: now also U$5.E1
- net EXT2: now also U$5.E2
- net EXT3: now also U$5.E3
- net EXT4: now also U$5.E4
- net EXT5: now also U$5.E5
- net EXT6: now also U$5.E6
- net EXT7: now also U$5.E7
- net GND: now also C54.1, C61.1, C63.1, IC13G$3.GND, R62A.2, R63A.2, R65A.2, R66A.2, U$5.GND@1, U$5.GND@2, U$8.GND@1, U$8.GND@2, U$9.SLEEVE; no longer U$2.2
- net GREEN: now also R59A.2
- net GREEN0: now also U$8.E5; no longer U$2.8
- net GREEN1: now also U$8.E4; no longer U$2.7
- net HSYNC: now also U$8.E0; no longer U$2.3
- net N$55: now also U$8.+5V; no longer IC2.__IO_84, TP5.TP
- net RCV: now also IC2.__IO_56; no longer IC2.__IO_59
- net RED: now also R58A.2
- net RED0: now also U$8.E3; no longer U$2.6
- net RED1: now also U$8.E2; no longer U$2.5
- net USB_FLT: now also IC2.__IO_62; no longer IC2.__IO_65
- net USB_MODE: now also IC2.__IO_58; no longer IC2.__IO_61
- net USB_OE: now also IC2.__IO_57; no longer IC2.__IO_60
- net USB_PWREN: now also IC2.__IO_63; no longer IC2.__IO_66
- net USB_SUSPEND: now also IC2.__IO_53; no longer IC2.__IO_56
- net VM: now also IC2.__IO_54; no longer IC2.__IO_57
- net VMO: now also IC2.__IO_61; no longer IC2.__IO_64
- net VP: now also IC2.__IO_55; no longer IC2.__IO_58
- net VPO: now also IC2.__IO_60; no longer IC2.__IO_63
- net VSYNC: now also U$8.E1; no longer U$2.4
Other:
- moved on the sheet: R53, R54, R55, R56, U$7

Commit message: r2.2 updates
Parts:
- added JP1: (no value), SparkFun-Connectors:PINHD-2X10
- added U$2: INTERFACEZ_EDGEDAUGHTER, alvie:INTERFACEZ_EDGEDAUGHTER
- R51, R53, R55: value 520R -> 1K24
- R52, R54, R56: value 270R -> 619R
- R58: value 520R -> 309R
- R59, R60: value 270R -> 309R
Connections:
- new net N$61: U$2.+5V
- net +3V3: now also U$2.+3V3
- net AUDIO_L: now also U$2.E11
- net AUDIO_R: now also U$2.E12
- net BLUE0: now also U$2.E7
- net BLUE1: now also U$2.E6
- net BLUE2: now also U$2.E8
- net GND: now also U$2.GND@1, U$2.GND@2
- net GREEN0: now also U$2.E5
- net GREEN1: now also U$2.E4
- net GREEN2: now also U$2.E10
- net HSYNC: now also U$2.E0
- net RED0: now also U$2.E3
- net RED1: now also U$2.E2
- net RED2: now also U$2.E9
- net VSYNC: now also U$2.E1
Other:
- note added: "Expansion"
- note added: "T10N"
- note added: "T10P"
- note added: "T11N"
- note added: "T11P"
- note added: "T12N"
- note added: "T12P"
- note added: "T16N"
- note added: "T16P"
- moved on the sheet: U$7

Commit message: Rev 2.2 for board
Parts:
- added C100, C101, C93, C94, C95: 100nF, GadgetFactory:C0603
- added C64, C66: 100nF 6.3V, GadgetFactory:C0603
- added C65: 47uF 6.3V TANT, alvie:TANT_CASE_A
- added C96: 2.2uF, GadgetFactory:C0805
- added C97: 1uF, GadgetFactory:C0603
- added C98: 1nF, GadgetFactory:C0603
- added C99: 100nF/DNP, GadgetFactory:C0603
- added IC14: LAN8720A, sigedi-footprints:LAN8720A
- added L8: 600R, GadgetFactory:L0805
- added R69, R70, R71, R79, R80: 2K2, GadgetFactory:R0603
- added R78: 10K, GadgetFactory:R0603
- added R81: 0R, GadgetFactory:R0603
- added R82: 12K1, GadgetFactory:R0603
- added R83, R84, R85, R86: 49R9, GadgetFactory:R0603
- added R87, R88: 330R, GadgetFactory:R0603
- added T1: Hanrun HR917550A, alvie:HR913550A
- added U$10: INTERFACEZ_EDGEDAUGHTER, alvie:INTERFACEZ_EDGEDAUGHTER
- added U$11, U$6: PMS150C-U06, alvie:PMS150C-U06
- added U$15: PIN-2X5-1.27MM, alvie:PIN-2X5-1.27MM
- added U$16: PIN-2X5, alvie:PIN-2X5
Connections:
- new net CLKIN: R81A.1, U$10.E0
- new net ETHID: R71A.1, U$10.E13, U$11.PA6
- new net ETH_CLK: IC14.XTAL1/CLKIN, R81A.2
- new net ETH_CRS_DV: IC14.CRS_DV/MODE2, U$10.E3
- new net ETH_MDC: IC14.MDC, R79A.1, U$10.E9
- new net ETH_MDIO: IC14.MDIO, R80A.1, U$10.E10
- new net ETH_NRST: IC14.NRST, R78A.1, U$10.E8
- new net ETH_REF_CLK: IC14.NINT/REFCLK0, U$10.E4
- new net ETH_RXD0: IC14.RXD0/MODE0, U$10.E2
- new net ETH_RXD1: IC14.RXD1/MODE1, U$10.E1
- new net ETH_RXERR: IC14.RXERR/PHYAD0, U$10.E11
- new net ETH_TXD0: IC14.TXD0, U$10.E7
- new net ETH_TXD1: IC14.TXD1, U$10.E6
- new net ETH_TX_EN: IC14.TXEN, U$10.E5
- new net EXTID: JP1.8, R70A.1, U$2.E13
- new net N$64: C101.1, T1G$1.5
- new net N$65: C100.1, T1G$1.4
- new net N$66: JP1.7, U$2.E0
- new net N$69: JP1.9, U$2.E1
- new net N$70: JP1.11, U$2.E2
- new net N$71: JP1.13, U$2.E3
- new net N$72: JP1.15, U$2.E4
- new net N$73: JP1.17, U$2.E5
- new net N$74: JP1.19, U$2.E6
- new net N$75: C99.2, L8.2, R83A.2, R84A.2, R85A.2, R86A.2
- new net N$76: R87A.2, T1YELLOW.K
- new net N$77: JP1.10, U$2.E12
- new net N$78: JP1.12, U$2.E11
- new net N$79: JP1.14, U$2.E10
- new net N$80: JP1.16, U$2.E9
- new net N$81: JP1.18, U$2.E8
- new net N$82: JP1.20, U$2.E7
- new net N$83: R88A.2, T1GREEN.K
- new net N$84: IC14.RBIAS, R82A.2
- new net N$85: C97.2, C98.2, IC14.VDDCR
- new net N$86: U$15.1, U$16.1
- new net N$87: U$15.3, U$16.3
- new net N$88: U$15.5, U$16.5
- new net N$89: U$15.7, U$16.7
- new net N$90: U$15.9, U$16.9
- new net N$91: U$15.2, U$16.2
- new net N$92: U$15.4, U$16.4
- new net N$93: U$15.6, U$16.6
- new net N$94: U$15.8, U$16.8
- new net N$95: U$15.10, U$16.10
- new net NC: U$10.+5V
- new net PHY_LED0: IC14.LED1/REGOFF, T1YELLOW.A
- new net PHY_LED1: IC14.LED2/NINTSEL, T1GREEN.A
- new net RXM: IC14.TXN, R84A.1, T1G$1.2
- new net RXP: IC14.TXP, R83A.1, T1G$1.1
- new net TXM: IC14.RXN, R86A.1, T1G$1.6
- new net TXP: IC14.RXP, R85A.1, T1G$1.3
- new net VGAID: R69A.1, U$6.PA6, U$8.E13
- net +3V3: now also C64.2, C65.+, C66.2, C93.2, C94.2, C95.2, C96.2, IC14.VDD1A, IC14.VDD2A, IC14.VDDIO, JP1.1, L8.1, R69A.2, R70A.2, R71A.2, R78A.2, R79A.2, R80A.2, U$10.+3V3, U$11.VCC, U$6.VCC
- net AUDIO_L: no longer U$2.E11
- net AUDIO_R: no longer U$2.E12
- net BLUE0: no longer U$2.E7
- net BLUE1: no longer U$2.E6
- net BLUE2: no longer U$2.E8
- net GND: now also C100.2, C101.2, C64.1, C65.-, C66.1, C93.1, C94.1, C95.1, C96.1, C97.1, C98.1, C99.1, IC14.VSS, JP1.3, JP1.4, R82A.1, R87A.1, R88A.1, U$10.GND@1, U$10.GND@2, U$11.GND, U$6.GND
- net GREEN0: no longer U$2.E5
- net GREEN1: no longer U$2.E4
- net GREEN2: no longer U$2.E10
- net HSYNC: no longer U$2.E0
- net N$61: now also JP1.2
- net PE: now also T1G$1.8, T1G$4.SHIELD
- net RED0: no longer U$2.E3
- net RED1: no longer U$2.E2
- net RED2: no longer U$2.E9
- net VSYNC: no longer U$2.E1
Other:
- moved on the sheet: JP1

Commit message: New tape structure
Other:
- note removed: "CHANGE TO PS!"
- note removed: "IO2 NEEDS PULLDOWN FOR SERIAL PROG!"
- note removed: "USB Host connector"
- moved on the sheet: C3, C31, C32, C33, C34, C37, C40, C41, C44, C48, C49, C51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

Commit message: Cosmetic changes
Other:
- note added: "FPGA"
- note added: "JTAG"
- note added: "QSPI SDRAM"
- note removed: "DMC3400SDW-7"
- note removed: "FPGA, Config Flash and JTAG"
- note removed: "SDRAM"
- moved on the sheet: C60, J1A, J1B, R10, R24, R25, R26, R8, R9

Commit message: Fix signal naming
Connections:
- net EXT10: now also IC2.__IO_66, U$5.E10; no longer IC2.__IO_65, U$5.E9
- net EXT11: now also IC2.__IO_67, U$5.E11; no longer IC2.__IO_64, U$5.E8
- net EXT8: now also IC2.__IO_64, U$5.E8; no longer IC2.__IO_67, U$5.E11
- net EXT9: now also IC2.__IO_65, U$5.E9; no longer IC2.__IO_66, U$5.E10
Changed lines of the file:
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@@
 </segment>
 </net>
-<net name="EXT8" class="0">
+<net name="EXT11" class="0">
 <segment>
 <pinref part="IC2" gate="G$1" pin="__IO_67"/>
@@
 </segment>
 </net>
-<net name="EXT9" class="0">
+<net name="EXT10" class="0">
 <segment>
 <pinref part="IC2" gate="G$1" pin="__IO_66"/>
@@
 </segment>
 </net>
-<net name="EXT10" class="0">
+<net name="EXT9" class="0">
 <segment>
 <pinref part="IC2" gate="G$1" pin="__IO_65"/>
@@
 </segment>
 </net>
-<net name="EXT11" class="0">
+<net name="EXT8" class="0">
 <segment>
 <pinref part="IC2" gate="G$1" pin="__IO_64"/>
