File: pcb/interfacez_main_r2_5.brd (EAGLE design)
At the start: 86 x 61 mm, 170 parts, among them IC1 STMPS2141STR, IC10 74LCX245FT, IC11 74LCX245FT, IC12 USB1T11AMTCX, IC13 74LVC06APW,118, IC2 EP4CE6E22C8N, IC3 74LCX245FT, IC4 74LCX245FT, IC5 74AHC1G125DCK, IC7 CH330N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

Commit message: pcb: update rev 2.5
Parts:
- removed R55: 140K, GadgetFactory:0603
- added R14: 0R, GadgetFactory:0603
- added TP2: TPTP12SQ, testpad:TP12SQ
- R1: value 8K66 1% -> 4K99 1%
- R24, R38: value 140K -> 47K
- R26: value 13K 1% -> 10K 1%
- R44: value 39K1 1% -> 31K6 1%
- R49: value 20R -> 33R
- moved R12 1.75 mm to (33.9, 22.6)
- moved Q6 1.00 mm to (18.3, 24.1)
- moved USB2 1.00 mm to (76.5, 53.0)
- moved R37 0.95 mm to (79.7, 39.1)
- moved C24 0.50 mm to (34.1, 18.9)
- moved IC10 0.50 mm to (38.2, 18.1)
- moved RN3 0.50 mm to (34.5, 13.1)
- moved R33 0.45 mm to (15.8, 24.0)
- renumbered U$2 to IC6, U$4 to IC14
Connections:
- new net N$1: Q5.3, R14.2
- new net N$19: IC2.8, TP2.TP
- net +9V: no longer R55.1
- net GND: no longer R55.2
- net IO6: now also IC2.25; no longer IC2.8
- net ROMCS2: now also R14.1; no longer Q5.3
Routing:
- net IO6: track 44.4 -> 51.5 mm
- net N$19: track 0.00 -> 4.09 mm
- net +5V: track 208.2 -> 212.0 mm, vias 16 -> 15
- net ROMCS2: track 57.7 -> 61.5 mm
- net PE: track 215.3 -> 218.4 mm
- net N$1: track 0.00 -> 2.59 mm
- net +3V3: track 558.2 -> 560.4 mm
- net A5: track 14.7 -> 12.9 mm
- net N$52: track 12.2 -> 14.0 mm
- net A6: track 15.9 -> 14.3 mm
- net CK_OUT_NEN: track 66.0 -> 67.1 mm
- net VBUS: track 24.0 -> 25.0 mm
- net DP: track 13.8 -> 14.8 mm
- net DM: track 13.5 -> 14.5 mm
- net N$62: track 1.35 -> 2.35 mm
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