File: pcb/interfacez_main_r2_5.sch (EAGLE design)
At the start: 167 parts, among them IC1 STMPS2141STR, IC10 74LCX245FT, IC11 74LCX245FT, IC12 USB1T11AMTCX, IC13 74LVC06APW,118, IC2 EP4CE6E22C8N, IC3 74LCX245FT, IC4 74LCX245FT, IC5 74AHC1G125DCK, IC7 CH330N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

Commit message: pcb: update rev 2.5
Parts:
- removed R55: 140K, GadgetFactory:R0603
- added R14: 0R, GadgetFactory:R0603
- added TP2: TPTP12SQ, testpad:TPTP12SQ
- R1: value 8K66 1% -> 4K99 1%
- R24, R38: value 140K -> 47K
- R26: value 13K 1% -> 10K 1%
- R44: value 39K1 1% -> 31K6 1%
- R49: value 20R -> 33R
- renumbered U$2 to IC6, U$4 to IC14
Connections:
- new net N$1: Q5T1.D, R14A.2
- new net N$19: IC2.__IO_6/FLASH_NCS/NCSO, TP2.TP
- net +9V: no longer R55A.1
- net GND: no longer R55A.2
- net IO6: now also IC2.__CLK3; no longer IC2.__IO_6/FLASH_NCS/NCSO
- net ROMCS2: now also R14A.1; no longer Q5T1.D
Other:
- note added: "Alt: RT6212BHGJ6F R1=12K, R99=24K,L1=2.2uH"
- note added: "Alt: RT6212BHGJ6F R1=75K, R99=24K,L1=3.6uH"
- note added: "Remove resistor if B4 is use for other purposes (i.e., audio in)"
